File: PCB/2 Layer nvme Carrier/HDMI.kicad_sch (KiCad schematic)
At the start: 37 parts, among them J4 HDMI_A, Q1 2N7002, Q2 2SK3018, Q3 2SK3018, Q4 2SK3018, U1 TPAZ1023-04F, U2 TPAZ1023-04F

Commit message: Parts change for BOM
Parts:
- C17, C18, C19, C20, C21, C22, C23, C24, C25: Mfr.# (none) -> GRM155R71H104KE14D
- D1, D2, D3: Mfr.# (none) -> ESD5V0B03-1006
- D4: Mfr.# (none) -> 1N5819WS
- F1: Mfr.# (none) -> 0603L050/6AR
- J4: Mfr.# (none) -> 2086581001
- Q1: Mfr.# (none) -> NDS7002A
- Q2, Q3, Q4: Mfr.# (none) -> 2SK3018
- R10, R13, R14, R16, R17, R7, R8, R9: Mfr.# (none) -> RC0402FR-07470RL
- R11: Mfr.# (none) -> RC0402FR-071KL
- R15, R18, R19, R3, R5: Mfr.# (none) -> RC0402FR-072K2L
- R4: Mfr.# (none) -> RC0402FR-071ML
- R6: Mfr.# (none) -> RC0402FR-0721K5L
- U1, U2: Mfr.# (none) -> TPAZ1023-04F

Commit message: BOM update and pdf
Parts:
- C17, C18, C19, C20, C21, C22, C23, C24, C25: MPN (none) -> GRM155R71H104KE14D; Mfr.# GRM155R71H104KE14D -> (none)
- D1, D2, D3: MPN (none) -> ESD5V0B03-1006; Mfr.# ESD5V0B03-1006 -> (none)
- D4: MPN (none) -> 1N5819WS; Mfr.# 1N5819WS -> (none)
- F1: MPN (none) -> 0603L050/6AR; Mfr.# 0603L050/6AR -> (none)
- J4: MPN (none) -> 2086581001; Mfr.# 2086581001 -> (none)
- Q1: MPN (none) -> NDS7002A; Mfr.# NDS7002A -> (none)
- Q2, Q3, Q4: MPN (none) -> 2SK3018; Mfr.# 2SK3018 -> (none)
- R10, R13, R14, R16, R17, R7, R8, R9: MPN (none) -> RC0402FR-07470RL; Mfr.# RC0402FR-07470RL -> (none)
- R11: MPN (none) -> RC0402FR-071KL; Mfr.# RC0402FR-071KL -> (none)
- R15, R18, R19, R3, R5: MPN (none) -> RC0402FR-072K2L; Mfr.# RC0402FR-072K2L -> (none)
- R4: MPN (none) -> RC0402FR-071ML; Mfr.# RC0402FR-071ML -> (none)
- R6: MPN (none) -> RC0402FR-0721K5L; Mfr.# RC0402FR-0721K5L -> (none)
- U1, U2: MPN (none) -> TPAZ1023-04F; Mfr.# TPAZ1023-04F -> (none)
