File: PCB/2 Layer nvme Carrier/PCIe.kicad_sch (KiCad schematic)
At the start: 22 parts, among them J200 Bus_PCI_Express_x4, J300 Bus_PCI_Express_x4

Commit message: Parts change for BOM
Parts:
- C201, C202, C301, C302: Mfr.# (none) -> GRM155R61H224KE01D
- C203, C204, C207, C209, C303, C304, C307, C309: Mfr.# (none) -> GRM155R71H104KE14D
- C205, C206, C305, C306: Mfr.# (none) -> PM101M025E077PTR
- C208, C308: Mfr.# (none) -> CL05A106MP5NUNC
- C210, C310: value 560uF/25V -> 470uF/10V; Mfr.# (none) -> VZT471M1ATR-0607
- J200, J300: Mfr.# (none) -> AAA-PCI-161-K03

Commit message: BOM update and pdf
Parts:
- C201, C202, C301, C302: MPN (none) -> GRM155R61H224KE01D; Mfr.# GRM155R61H224KE01D -> (none)
- C203, C204, C207, C209, C303, C304, C307, C309: MPN (none) -> GRM155R71H104KE14D; Mfr.# GRM155R71H104KE14D -> (none)
- C205, C206, C305, C306: MPN (none) -> PM101M025E077PTR; Mfr.# PM101M025E077PTR -> (none)
- C208, C308: MPN (none) -> CL05A106MP5NUNC; Mfr.# CL05A106MP5NUNC -> (none)
- C210, C310: MPN (none) -> VZT471M1ATR-0607; Mfr.# VZT471M1ATR-0607 -> (none)
- J200, J300: MPN (none) -> AAA-PCI-161-K03; Mfr.# AAA-PCI-161-K03 -> (none)

Commit message: change to 12V and more work to do
Parts:
- J200, J300: MPN_alt (none) -> 2EG03227-D2D-DF
Connections:
- net +12VA renamed +12V
Changed lines of the file:
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@@
 		(on_board yes)
 		(dnp no)
-		(fields_autoplaced yes)
 		(property "Reference" "#PWR0150"
 			(at 335.28 162.56 0)
@@
 			)
 		)
-		(property "Value" "+12VA"
-			(at 335.28 153.67 0)
-			(effects
-				(font
-					(size 1.27 1.27)
-				)
+		(property "Value" "+12V"
+			(at 333.502 154.178 0)
+			(effects
+				(font
+					(size 1.27 1.27)
+				)
+				(justify left)
 			)
 		)
@@
 		)
 		(property "MPN" "AAA-PCI-161-K03"
+			(at 369.57 214.63 0)
+			(effects
+				(font
+					(size 1.27 1.27)
+				)
+				(hide yes)
+			)
+		)
+		(property "MPN_alt" "2EG03227-D2D-DF"
 			(at 369.57 214.63 0)
 			(effects
@@
 			)
 		)
+		(property "MPN_alt" "2EG03227-D2D-DF"
+			(at 184.15 213.36 0)
+			(effects
+				(font
+					(size 1.27 1.27)
+				)
+				(hide yes)
+			)
+		)
 		(pin "A1"
 		)
@@
 		(on_board yes)
 		(dnp no)
-		(fields_autoplaced yes)
 		(property "Reference" "#PWR013"
 			(at 149.86 161.29 0)
@@
 			)
 		)
-		(property "Value" "+12VA"
-			(at 149.86 152.4 0)
-			(effects
-				(font
-					(size 1.27 1.27)
-				)
-			)
-		)
+		(property "Value" "+12V"
+			(at 148.082 153.416 0)
+			(effects
+				(font
+					(size 1.27 1.27)
+				)
+				(justify left)
+			)
+		)
