File: PCB/2 Layer nvme Carrier/fan_temp.kicad_sch (KiCad schematic)
At the start: 20 parts, among them M1 Fan_4pin, M2 Fan_4pin

Commit message: Parts change for BOM
Parts:
- C84, C85: Mfr.# (none) -> GRM155R71H104KE14D
- D26: Mfr.# (none) -> 1N5819WS
- D27: footprint Diode_SMD:D_SOD-323 -> A_HDJ_Library:D_SOD-323; Mfr.# (none) -> 1N5819WS
- M1: Mfr.# (none) -> B4B-PH-K-S-GW
- M2: footprint Connector_JST:JST_PH_B4B-PH-K_1x04_P2.00mm_Vertical -> Connector:FanPinHeader_1x04_P2.54mm_Vertical; Mfr.# (none) -> 470531000
- R67, R68, R70: Mfr.# (none) -> RC0402FR-0721K5L
- R69, R71: Mfr.# (none) -> RC0402FR-07100RL
- R72, R74: Mfr.# (none) -> RC0402FR-074K7L

Commit message: BOM update and pdf
Parts:
- C84, C85: MPN (none) -> GRM155R71H104KE14D; Mfr.# GRM155R71H104KE14D -> (none)
- D26, D27: MPN (none) -> 1N5819WS; Mfr.# 1N5819WS -> (none)
- M1: MPN (none) -> B4B-PH-K-S-GW; Mfr.# B4B-PH-K-S-GW -> (none)
- M2: MPN (none) -> 470531000; Mfr.# 470531000 -> (none)
- R67, R68, R70: MPN (none) -> RC0402FR-0721K5L; Mfr.# RC0402FR-0721K5L -> (none)
- R69, R71: MPN (none) -> RC0402FR-07100RL; Mfr.# RC0402FR-07100RL -> (none)
- R72, R74: MPN (none) -> RC0402FR-074K7L; Mfr.# RC0402FR-074K7L -> (none)
Changed lines of the file:
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@@
 	(title_block
 		(title "nvme Carrier for LattePanda Mu")
-		(date "2024-05-24")
-		(rev "V1.0.6")
+		(date "2024-07-13")
+		(rev "V1.0")
 	)
 	(junction
@@
 			)
 		)
-		(property "Mfr.# " ""
-			(at 332.74 167.64 0)
-			(effects
-				(font
-					(size 1.27 1.27)
-				)
-				(hide yes)
-			)
-		)
 		(property "Part#" ""
 			(at 332.74 167.64 0)
@@
 			)
 		)
-		(property "Mfr.#" "RC0402FR-07100RL"
+		(property "MPN" "RC0402FR-07100RL"
 			(at 332.74 167.64 0)
 			(effects
@@
 			)
 		)
-		(property "Mfr.# " ""
-			(at 332.74 243.84 0)
-			(effects
-				(font
-					(size 1.27 1.27)
-				)
-				(hide yes)
-			)
-		)
 		(property "Part#" ""
 			(at 332.74 243.84 0)
@@
 			)
 		)
-		(property "Mfr.#" "RC0402FR-07100RL"
+		(property "MPN" "RC0402FR-07100RL"
 			(at 332.74 243.84 0)
 			(effects
@@
 			)
 		)
-		(property "Mfr.# " ""
-			(at 213.36 158.75 0)
-			(effects
-				(font
-					(size 1.27 1.27)
-				)
-				(hide yes)
-			)
-		)
 		(property "Part#" ""
 			(at 213.36 158.75 0)
@@
 			)
 		)
-		(property "Mfr.# " ""
-			(at 313.69 173.99 0)
-			(effects
-				(font
-					(size 1.27 1.27)
-				)
-				(hide yes)
-			)
-		)
 		(property "Part#" ""
 			(at 313.69 173.99 0)
@@
 			)
 		)
-		(property "Mfr.# " ""
-			(at 226.06 165.1 0)
-			(effects
-				(font
-					(size 1.27 1.27)
-				)
-				(hide yes)
-			)
-		)
 		(property "Part#" ""
 			(at 226.06 165.1 0)
@@
 			)
 		)
-		(property "Mfr.# " ""
-			(at 341.63 151.13 0)
-			(effects
-				(font
-					(size 1.27 1.27)
-				)
-				(hide yes)
-			)
-		)
 		(property "Part#" ""
 			(at 341.63 151.13 0)
@@
 			)
 		)
-		(property "Mfr.#" "GRM155R71H104KE14D"
+		(property "MPN" "GRM155R71H104KE14D"
 			(at 341.63 151.13 0)
 			(effects
@@
 			)
 		)
-		(property "Mfr.# " ""
-			(at 391.16 241.3 0)
-			(effects
-				(font
-					(size 1.27 1.27)
-				)
-				(hide yes)
-			)
-		)
 		(property "Part#" ""
 			(at 391.16 241.3 0)
@@
 			)
 		)
-		(property "Mfr.#" "470531000"
+		(property "MPN" "470531000"
 			(at 391.16 241.3 0)
 			(effects
@@
 			)
 		)
-		(property "Mfr.# " ""
-			(at 365.76 228.6 0)
-			(effects
-				(font
-					(size 1.27 1.27)
-				)
-				(hide yes)
-			)
-		)
 		(property "Part#" ""
 			(at 365.76 228.6 0)
@@
 			)
 		)
-		(property "Mfr.#" "1N5819WS"
+		(property "MPN" "1N5819WS"
 			(at 365.76 228.6 0)
 			(effects
@@
 			)
 		)
-		(property "Mfr.# " ""
-			(at 341.63 227.33 0)
-			(effects
-				(font
-					(size 1.27 1.27)
-				)
-				(hide yes)
-			)
-		)
 		(property "Part#" ""
 			(at 341.63 227.33 0)
@@
 			)
 		)
-		(property "Mfr.#" "GRM155R71H104KE14D"
+		(property "MPN" "GRM155R71H104KE14D"
 			(at 341.63 227.33 0)
 			(effects
@@
 			)
 		)
-		(property "Mfr.# " ""
-			(at 302.26 152.4 0)
-			(effects
-				(font
-					(size 1.27 1.27)
-				)
-				(hide yes)
-			)
-		)
 		(property "Part#" ""
 			(at 302.26 152.4 0)
@@
 			)
 		)
-		(property "Mfr.# " ""
-			(at 332.74 238.76 0)
-			(effects
-				(font
-					(size 1.27 1.27)
-				)
-				(hide yes)
-			)
-		)
 		(property "Part#" ""
 			(at 332.74 238.76 0)
@@
 			)
 		)
-		(property "Mfr.#" "RC0402FR-0721K5L"
+		(property "MPN" "RC0402FR-0721K5L"
 			(at 332.74 238.76 0)
 			(effects
@@
 			)
 		)
-		(property "Mfr.#" "B4B-PH-K-S-GW"
-			(at 391.16 165.1 0)
-			(effects
-				(font
-					(size 1.27 1.27)
-				)
-				(hide yes)
-			)
-		)
-		(property "Mfr.# " ""
+		(property "Part#" ""
 			(at 391.16 165.1 0)
 			(effects
@@
 			)
 		)
-		(property "Part#" ""
+		(property "MPN" "B4B-PH-K-S-GW"
 			(at 391.16 165.1 0)
 			(effects
@@
 			)
 		)
-		(property "Mfr.# " ""
-			(at 302.26 228.6 0)
-			(effects
-				(font
-					(size 1.27 1.27)
-				)
-				(hide yes)
-			)
-		)
 		(property "Part#" ""
 			(at 302.26 228.6 0)
@@
 			)
 		)
-		(property "Mfr.# " ""
-			(at 332.74 162.56 0)
-			(effects
-				(font
-					(size 1.27 1.27)
-				)
-				(hide yes)
-			)
-		)
 		(property "Part#" ""
 			(at 332.74 162.56 0)
@@
 			)
 		)
-		(property "Mfr.#" "RC0402FR-0721K5L"
+		(property "MPN" "RC0402FR-0721K5L"
 			(at 332.74 162.56 0)
 			(effects
@@
 			)
 		)
-		(property "Mfr.# " ""
-			(at 226.06 152.4 0)
-			(effects
-				(font
-					(size 1.27 1.27)
-				)
-				(hide yes)
-			)
-		)
 		(property "Part#" ""
 			(at 226.06 152.4 0)
@@
 			)
 		)
-		(property "Mfr.# " ""
-			(at 313.69 250.19 0)
-			(effects
-				(font
-					(size 1.27 1.27)
-				)
-				(hide yes)
-			)
-		)
 		(property "Part#" ""
 			(at 313.69 250.19 0)
@@
 			)
 		)
-		(property "Mfr.#" "RC0402FR-0721K5L"
+		(property "MPN" "RC0402FR-0721K5L"
 			(at 313.69 250.19 0)
 			(effects
@@
 			)
 		)
-		(property "Mfr.# " ""
-			(at 365.76 152.4 0)
-			(effects
-				(font
-					(size 1.27 1.27)
-				)
-				(hide yes)
-			)
-		)
 		(property "Part#" ""
 			(at 365.76 152.4 0)
@@
 			)
 		)
-		(property "Mfr.#" "1N5819WS"
+		(property "MPN" "1N5819WS"
 			(at 365.76 152.4 0)
 			(effects
@@
 			)
 		)
-		(property "Mfr.# " ""
-			(at 353.06 228.6 0)
-			(effects
-				(font
-					(size 1.27 1.27)
-				)
-				(hide yes)
-			)
-		)
 		(property "Part#" ""
 			(at 353.06 228.6 0)
@@
 			)
 		)
-		(property "Mfr.#" "RC0402FR-074K7L"
+		(property "MPN" "RC0402FR-074K7L"
 			(at 353.06 228.6 0)
 			(effects
@@
 			)
 		)
-		(property "Mfr.# " ""
-			(at 353.06 152.4 0)
-			(effects
-				(font
-					(size 1.27 1.27)
-				)
-				(hide yes)
-			)
-		)
 		(property "Part#" ""
 			(at 353.06 152.4 0)
@@
 			)
 		)
-		(property "Mfr.#" "RC0402FR-074K7L"
+		(property "MPN" "RC0402FR-074K7L"
 			(at 353.06 152.4 0)
 			(effects
@@
 			(at 353.06 215.9 0)
 			(effects
-				(font
-					(size 1.27 1.27)
-				)
-				(hide yes)
-			)
-		)
-		(property "Mfr.# " ""
-			(at 353.06 215.9 0)
-			(effects

Commit message: change to 12V and more work to do
Connections:
- net +12VA renamed +12V
Changed lines of the file:
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@@
 		(on_board yes)
 		(dnp no)
-		(fields_autoplaced yes)
 		(property "Reference" "#PWR0116"
 			(at 365.76 215.9 0)
@@
 			)
 		)
-		(property "Value" "+12VA"
-			(at 365.76 207.01 0)
+		(property "Value" "+12V"
+			(at 362.966 207.264 0)
 			(effects
 				(font
 					(size 1.27 1.27)
 				)
+				(justify left)
 			)
 		)
