File: PCB/2 Layer nvme Carrier/M.2 M Key.kicad_sch (KiCad schematic)
At the start: 85 parts, among them J100 Bus_M.2_Socket_M, J110 Bus_M.2_Socket_M, J120 Bus_M.2_Socket_M, J130 Bus_M.2_Socket_M, J140 Bus_M.2_Socket_M, J150 Bus_M.2_Socket_M

Commit message: Parts change for BOM
Parts:
- C101, C103, C111, C113, C121, C123, C131, C133, C141, C143, C151, C153: Mfr.# (none) -> CL05A106MP5NUNC
- C102, C104, C112, C114, C122, C124, C132, C134, C142, C144, C152, C154: Mfr.# (none) -> GRM155R71H104KE14D
- C105, C106, C115, C116, C125, C126, C135, C136, C145, C146, C155, C156: Mfr.# (none) -> GRM155R61H224KE01D
- D101, D111, D121, D131, D141, D151: Mfr.# (none) -> SZYY0603YG
- H1032, H1042, H1060, H1080, H1130, H1142, H1160, H1180, H1230, H1242, H1260, H1280, H1330, H1342, H1360, H1380, H1430, H1442, H1460, H1480, H1530, H1542, H1560, H1580: value MountingHole_M2.0 -> MountingHole_M2.5
- J100, J110, J120, J130, J140, J150: Mfr.# (none) -> 1-2199230-5
- R102, R112, R122, R132, R142, R152: Mfr.# (none) -> RC0402FR-072K2L
- R103, R113, R123, R133, R143, R153: Mfr.# (none) -> RMC 0402 0R N

Commit message: BOM update and pdf
Parts:
- C101, C103, C111, C113, C121, C123, C131, C133, C141, C143, C151, C153: MPN (none) -> CL05A106MP5NUNC; Mfr.# CL05A106MP5NUNC -> (none)
- C102, C104, C112, C114, C122, C124, C132, C134, C142, C144, C152, C154: MPN (none) -> GRM155R71H104KE14D; Mfr.# GRM155R71H104KE14D -> (none)
- C105, C106, C115, C116, C125, C126, C135, C136, C145, C146, C155, C156: MPN (none) -> GRM155R61H224KE01D; Mfr.# GRM155R61H224KE01D -> (none)
- D101, D111, D121, D131, D141, D151: MPN (none) -> SZYY0603YG; Mfr.# SZYY0603YG -> (none)
- J100, J110, J120, J130, J140, J150: MPN (none) -> 1-2199230-5; Mfr.# 1-2199230-5 -> (none)
- R102, R112, R122, R132, R142, R152: MPN (none) -> RC0402FR-072K2L; Mfr.# RC0402FR-072K2L -> (none)
- R103, R113, R123, R133, R143, R153: MPN (none) -> RMC 0402 0R N; Mfr.# RMC 0402 0R N -> (none)

Commit message: Rework for PSU and REFCLK
Parts:
- removed R103, R113, R123, R133, R143, R153: 0R/1%, A_HDJ_Library:R_0402_1005Metric, symbol Device:R
- removed R134: 0R/1%, Resistor_SMD:R_0402_1005Metric, symbol Device:R
Connections:
- removed net CLKREQB: J130.52 (~{CLKREQ}), J140.52 (~{CLKREQ}), J150.52 (~{CLKREQ})
- removed net CLKREQF: J100.52 (~{CLKREQ}), J110.52 (~{CLKREQ}), J120.52 (~{CLKREQ})
- removed net REFCLKMB+: J130.55 (REFCLKp), J140.55 (REFCLKp), J150.55 (REFCLKp)
- removed net REFCLKMB-: J130.53 (REFCLKn), J140.53 (REFCLKn), J150.53 (REFCLKn)
- removed net REFCLKMF+: J100.55 (REFCLKp), J110.55 (REFCLKp), J120.55 (REFCLKp)
- removed net REFCLKMF-: J100.53 (REFCLKn), J110.53 (REFCLKn), J120.53 (REFCLKn)
- removed net ~{WAKE}: J100.54 (~{PEWAKE}), J110.54 (~{PEWAKE}), J120.54 (~{PEWAKE}), J130.54 (~{PEWAKE}), J140.54 (~{PEWAKE}), J150.54 (~{PEWAKE})
- new net CLKREQ3: J100.52 (~{CLKREQ})
- new net CLKREQ4: J110.52 (~{CLKREQ})
- new net REFCLKM2a+: J120.55 (REFCLKp)
- new net REFCLKM2a-: J120.53 (REFCLKn)
- new net REFCLKM2b+: J130.55 (REFCLKp)
- new net REFCLKM2b-: J130.53 (REFCLKn)
- new net REFCLKM2c+: J140.55 (REFCLKp)
- new net REFCLKM2c-: J140.53 (REFCLKn)
- new net REFCLKM3+: J100.55 (REFCLKp)
- new net REFCLKM3-: J100.53 (REFCLKn)
- new net REFCLKM3c+: J150.55 (REFCLKp)
- new net REFCLKM3c-: J150.53 (REFCLKn)
- new net REFCLKM4+: J110.55 (REFCLKp)
- new net REFCLKM4-: J110.53 (REFCLKn)
- no-connect marks 83 -> 100
Other:
- note removed: "32.768kHz clock for low power mode"
- note removed: "To be grounded for SATA, No Connect for PCIe"

Commit message: Rework started with PCIe
Connections:
- net ~{WAKE}: now reaches J100.54 (~{PEWAKE})
- net ~{WAKE}: now also J110.54 (~{PEWAKE}), J120.54 (~{PEWAKE}), J130.54 (~{PEWAKE}), J140.54 (~{PEWAKE}), J150.54 (~{PEWAKE})
- net CLKREQM3: now reaches J150.52 (~{CLKREQ})
- net CLKREQM1: now reaches J130.52 (~{CLKREQ})
- net CLKREQM2: now reaches J140.52 (~{CLKREQ})
- net CLKREQM0: now reaches J120.52 (~{CLKREQ})
- no-connect marks 100 -> 90

Commit message: PCIe and CLK Buffenr Lines
Connections:
- net CLKREQ3 is gone; now on net CLKREQM0: J100.52 (~{CLKREQ})
- net CLKREQ4 is gone; now on net CLKREQM1: J110.52 (~{CLKREQ})
- net REFCLKM2b+ is gone; now on net REFCLKM3+: J130.55 (REFCLKp)
- net REFCLKM2b- is gone; now on net REFCLKM3-: J130.53 (REFCLKn)
- net REFCLKM2c+ is gone; now on net REFCLKM4+: J140.55 (REFCLKp)
- net REFCLKM2c- is gone; now on net REFCLKM4-: J140.53 (REFCLKn)
- net CLKREQM0: no longer J120.52 (~{CLKREQ})
- net CLKREQM1: no longer J130.52 (~{CLKREQ})
- net CLKREQM2: now also J120.52 (~{CLKREQ}); no longer J140.52 (~{CLKREQ})
- net CLKREQM3: now also J130.52 (~{CLKREQ}); no longer J150.52 (~{CLKREQ})
- net REFCLKM3+: no longer J100.55 (REFCLKp)
- net REFCLKM3-: no longer J100.53 (REFCLKn)
- net REFCLKM4+: no longer J110.55 (REFCLKp)
- net REFCLKM4-: no longer J110.53 (REFCLKn)
- net REFCLKM2a+ renamed REFCLKM2+
- net REFCLKM2a- renamed REFCLKM2-
- net REFCLKM3c+ renamed REFCLKM5+
- net REFCLKM3c- renamed REFCLKM5-
- new net CLKREQM4: J140.52 (~{CLKREQ})
- new net CLKREQM5: J150.52 (~{CLKREQ})
- new net REFCLKM0+: J100.55 (REFCLKp)
- new net REFCLKM0-: J100.53 (REFCLKn)
- new net REFCLKM1+: J110.55 (REFCLKp)
- new net REFCLKM1-: J110.53 (REFCLKn)
