File: PCB/2 Layer nvme Carrier/USB.kicad_sch (KiCad schematic)
At the start: 18 parts, among them J2 USB_A_Stacked, J3 USB3_A, J78 USB_A, U3 ULC0524P, U4 ULC0524P

Commit message: Parts change for BOM
Parts:
- C28, C29: Mfr.# (none) -> GRM155R71H104KE14D
- C30, C32, C88: Mfr.# (none) -> CL10A226MP8NUNE
- D5, D6, D79, D80: Mfr.# (none) -> ESD5V0B03-1006
- F2, F3, F78: Mfr.# (none) -> BSMD0805-100-6V
- F5: Mfr.# (none) -> BSMD0805L-200
- J2: Mfr.# (none) -> UJ2-ADH-W1-TH
- J3: footprint Connector_USB:USB3_A_Molex_48393-001 -> Connector_USB:USB3_A_Receptacle_Wuerth_692122030100; Mfr.# (none) -> 692122030100
- J78: Mfr.# (none) -> 1050570001
- U3, U4: Mfr.# (none) -> ULC0524P

Commit message: BOM update and pdf
Parts:
- C28, C29: MPN (none) -> GRM155R71H104KE14D; Mfr.# GRM155R71H104KE14D -> (none)
- C30, C32, C88: MPN (none) -> CL10A226MP8NUNE; Mfr.# CL10A226MP8NUNE -> (none)
- D5, D6, D79, D80: MPN (none) -> ESD5V0B03-1006; Mfr.# ESD5V0B03-1006 -> (none)
- F2, F3, F78: MPN (none) -> BSMD0805-100-6V; Mfr.# BSMD0805-100-6V -> (none)
- F5: MPN (none) -> BSMD0805L-200; Mfr.# BSMD0805L-200 -> (none)
- J2: MPN (none) -> UJ2-ADH-W1-TH; Mfr.# UJ2-ADH-W1-TH -> (none)
- J3: MPN (none) -> 692122030100; Mfr.# 692122030100 -> (none)
- J78: MPN (none) -> 1050570001; Mfr.# 1050570001 -> (none)
- U3, U4: MPN (none) -> ULC0524P; Mfr.# ULC0524P -> (none)
Changed lines of the file:
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@@
 	(title_block
 		(title "nvme Carrier for LattePanda Mu")
-		(date "2024-05-24")
-		(rev "V1.0.6")
+		(date "2024-07-13")
+		(rev "V1.0")
 	)
 	(junction
@@
 			)
 		)
-		(property "Mfr.# " ""
-			(at 173.99 254 0)
-			(effects
-				(font
-					(size 1.27 1.27)
-				)
-				(hide yes)
-			)
-		)
 		(property "Part#" ""
 			(at 173.99 254 0)
@@
 			)
 		)
-		(property "Mfr.#" "ESD5V0B03-1006"
+		(property "MPN" "ESD5V0B03-1006"
 			(at 173.99 254 0)
 			(effects
@@
 			)
 		)
-		(property "Mfr.# " ""
-			(at 309.88 152.4 0)
-			(effects
-				(font
-					(size 1.27 1.27)
-				)
-				(hide yes)
-			)
-		)
 		(property "Part#" ""
 			(at 309.88 152.4 0)
@@
 			)
 		)
-		(property "Mfr.#" "BSMD0805-100-6V"
+		(property "MPN" "BSMD0805-100-6V"
 			(at 309.88 152.4 0)
 			(effects
@@
 			)
 		)
-		(property "Mfr.#" "ULC0524P"
-			(at 287.02 181.61 0)
-			(effects
-				(font
-					(size 1.27 1.27)
-				)
-				(hide yes)
-			)
-		)
-		(property "Mfr.# " ""
+		(property "Part#" ""
 			(at 287.02 181.61 0)
 			(effects
@@
 			)
 		)
-		(property "Part#" ""
+		(property "MPN" "ULC0524P"
 			(at 287.02 181.61 0)
 			(effects
@@
 			)
 		)
-		(property "Mfr.# " ""
-			(at 309.88 85.09 0)
-			(effects
-				(font
-					(size 1.27 1.27)
-				)
-				(hide yes)
-			)
-		)
 		(property "Part#" ""
 			(at 309.88 85.09 0)
@@
 			)
 		)
-		(property "Mfr.#" "BSMD0805-100-6V"
+		(property "MPN" "BSMD0805-100-6V"
 			(at 309.88 85.09 0)
 			(effects
@@
 			)
 		)
-		(property "Mfr.# " ""
-			(at 298.45 105.41 0)
-			(effects
-				(font
-					(size 1.27 1.27)
-				)
-				(hide yes)
-			)
-		)
 		(property "Part#" ""
 			(at 298.45 105.41 0)
@@
 			)
 		)
-		(property "Mfr.#" "ESD5V0B03-1006"
+		(property "MPN" "ESD5V0B03-1006"
 			(at 298.45 105.41 0)
 			(effects
@@
 			)
 		)
-		(property "Mfr.# " ""
-			(at 309.88 154.94 0)
-			(effects
-				(font
-					(size 1.27 1.27)
-				)
-				(hide yes)
-			)
-		)
 		(property "Part#" ""
 			(at 309.88 154.94 0)
@@
 			)
 		)
-		(property "Mfr.#" "BSMD0805-100-6V"
+		(property "MPN" "BSMD0805-100-6V"
 			(at 309.88 154.94 0)
 			(effects
@@
 			)
 		)
-		(property "Mfr.# " ""
-			(at 326.39 270.51 0)
-			(effects
-				(font
-					(size 1.27 1.27)
-				)
-				(hide yes)
-			)
-		)
 		(property "Part#" ""
 			(at 326.39 270.51 0)
@@
 			)
 		)
-		(property "Mfr.#" "692122030100"
+		(property "MPN" "692122030100"
 			(at 326.39 270.51 0)
 			(effects
@@
 			)
 		)
-		(property "Mfr.# " ""
-			(at 293.37 152.4 0)
-			(effects
-				(font
-					(size 1.27 1.27)
-				)
-				(hide yes)
-			)
-		)
 		(property "Part#" ""
 			(at 293.37 152.4 0)
@@
 			)
 		)
-		(property "Mfr.#" "CL10A226MP8NUNE"
+		(property "MPN" "CL10A226MP8NUNE"
 			(at 293.37 152.4 0)
 			(effects
@@
 			)
 		)
-		(property "Mfr.# " ""
-			(at 328.93 162.56 0)
-			(effects
-				(font
-					(size 1.27 1.27)
-				)
-				(hide yes)
-			)
-		)
 		(property "Part#" ""
 			(at 328.93 162.56 0)
@@
 			)
 		)
-		(property "Mfr.#" "UJ2-ADH-W1-TH"
+		(property "MPN" "UJ2-ADH-W1-TH"
 			(at 328.93 162.56 0)
 			(effects
@@
 			)
 		)
-		(property "Mfr.# " ""
-			(at 256.54 280.67 0)
-			(effects
-				(font
-					(size 1.27 1.27)
-				)
-				(hide yes)
-			)
-		)
 		(property "Part#" ""
 			(at 256.54 280.67 0)
@@
 			)
 		)
-		(property "Mfr.#" "GRM155R71H104KE14D"
+		(property "MPN" "GRM155R71H104KE14D"
 			(at 256.54 280.67 0)
 			(effects
@@
 			)
 		)
-		(property "Mfr.# " ""
-			(at 293.37 260.35 0)
-			(effects
-				(font
-					(size 1.27 1.27)
-				)
-				(hide yes)
-			)
-		)
 		(property "Part#" ""
 			(at 293.37 260.35 0)
@@
 			)
 		)
-		(property "Mfr.#" "CL10A226MP8NUNE"
+		(property "MPN" "CL10A226MP8NUNE"
 			(at 293.37 260.35 0)
 			(effects
@@
 			)
 		)
-		(property "Mfr.# " ""
-			(at 293.37 85.09 0)
-			(effects
-				(font
-					(size 1.27 1.27)
-				)
-				(hide yes)
-			)
-		)
 		(property "Part#" ""
 			(at 293.37 85.09 0)
@@
 			)
 		)
-		(property "Mfr.#" "CL10A226MP8NUNE"
+		(property "MPN" "CL10A226MP8NUNE"
 			(at 293.37 85.09 0)
 			(effects
@@
 			)
 		)
-		(property "Mfr.# " ""
-			(at 256.54 283.21 0)
-			(effects
-				(font
-					(size 1.27 1.27)
-				)
-				(hide yes)
-			)
-		)
 		(property "Part#" ""
 			(at 256.54 283.21 0)
@@
 			)
 		)
-		(property "Mfr.#" "GRM155R71H104KE14D"
+		(property "MPN" "GRM155R71H104KE14D"
 			(at 256.54 283.21 0)
 			(effects
@@
 			)
 		)
-		(property "Mfr.#" "ULC0524P"
-			(at 248.92 231.14 0)
-			(effects
-				(font
-					(size 1.27 1.27)
-				)
-				(hide yes)
-			)
-		)
-		(property "Mfr.# " ""
+		(property "Part#" ""
 			(at 248.92 231.14 0)
 			(effects
@@
 			)
 		)
-		(property "Part#" ""
+		(property "MPN" "ULC0524P"
 			(at 248.92 231.14 0)
 			(effects
@@
 			)
 		)
-		(property "Mfr.# " ""
-			(at 163.83 254 0)
-			(effects
-				(font
-					(size 1.27 1.27)
-				)
-				(hide yes)
-			)
-		)
 		(property "Part#" ""
 			(at 163.83 254 0)
@@
 			)
 		)
-		(property "Mfr.#" "ESD5V0B03-1006"
+		(property "MPN" "ESD5V0B03-1006"
 			(at 163.83 254 0)
 			(effects
@@
 			)
 		)
-		(property "Mfr.# " ""
-			(at 309.88 260.35 0)
-			(effects
-				(font
-					(size 1.27 1.27)
-				)
-				(hide yes)
-			)
-		)
 		(property "Part#" ""
 			(at 309.88 260.35 0)
@@
 			)
 		)
-		(property "Mfr.#" "BSMD0805L-200"
+		(property "MPN" "BSMD0805L-200"
 			(at 309.88 260.35 0)
 			(effects
@@
 			)
 		)
-		(property "Mfr.# " ""
-			(at 288.29 105.41 0)
-			(effects
-				(font
-					(size 1.27 1.27)
-				)
-				(hide yes)
-			)
-		)
 		(property "Part#" ""
 			(at 288.29 105.41 0)
@@
 			)
 		)
-		(property "Mfr.#" "ESD5V0B03-1006"
+		(property "MPN" "ESD5V0B03-1006"
 			(at 288.29 105.41 0)
 			(effects
@@
 			)
 		)
-		(property "Mfr.# " ""
-			(at 327.66 90.17 0)
-			(effects
-				(font
-					(size 1.27 1.27)
-				)
-				(hide yes)
-			)
-		)
 		(property "Part#" ""
 			(at 327.66 90.17 0)
@@
 			)
 		)
-		(property "Mfr.#" "1050570001"
+		(property "MPN" "1050570001"
 			(at 327.66 90.17 0)
 			(effects

Commit message: Work
Other:
- moved on the sheet: C28, C29, C30, C32, C88, D5, D6, D79, D80, F2, F3, F5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
