File: PCB/2 Layer nvme Carrier/nvme Carrier for LattePanda Mu.kicad_pcb (KiCad board)
At the start: 2 copper layers, 170.2 x 170.2 mm, 382 parts, among them J1 Conn_01x03_Pin, J100 Bus_M.2_Socket_M, J110 Bus_M.2_Socket_M, J120 Bus_M.2_Socket_M, J130 Bus_M.2_Socket_M, J140 Bus_M.2_Socket_M, J150 Bus_M.2_Socket_M, J2 USB_A_Stacked, J200 Bus_PCI_Express_x4, J3 USB3_A, J300 Bus_PCI_Express_x4, J4 HDMI_A, J481 Conn_01x02_Pin, J5 Barrel_Jack_Switch, J78 USB_A, J79 Conn_01x02_Pin, J80 Conn_01x02_Pin, J81 Conn_01x02_Pin, J82 Conn_01x04, M1 Fan_4pin, M2 Fan_4pin, Q1 2N7002, Q2 2SK3018, Q3 2SK3018, Q4 2SK3018, Q8 2N7002, SW1 SW_Push, SW2 SW_Push, U1 TPAZ1023-04F, U15 SY8253ADC, U16 SY8253ADC, U2 TPAZ1023-04F, U3 ULC0524P, U4 ULC0524P, U400 SY8253ADC, U410 SY8253ADC, U420 SY8253ADC, U430 SY8253ADC, U440 SY8253ADC, U450 SY8253ADC, U460 SY8253ADC, U480 SY8253ADC, U78 AMS1117-3.3, U79 W25Q128JVSIQ

Commit message: PCIe and CLK Buffenr Lines
Parts:
- removed J81: Conn_01x02_Pin, Connector_PinHeader_2.54mm:PinHeader_1x02_P2.54mm_Vertical
- added J11: Conn_01x03_Pin, Connector_PinHeader_2.54mm:PinHeader_1x03_P2.54mm_Vertical, F.Cu at (34.2, 85.2)
- added R95: 10K/1%, A_HDJ_Library:R_0402_1005Metric, F.Cu at (37.2, 85.2)
- added R96: 10K/1%, Resistor_SMD:R_0402_1005Metric, F.Cu at (139.0, 104.5)
- added R97: 10K/1%, Resistor_SMD:R_0402_1005Metric, F.Cu at (136.7, 104.5)
- added R98: 10K/1%, Resistor_SMD:R_0402_1005Metric, F.Cu at (132.0, 99.5)
- added R99: 10K/1%, Resistor_SMD:R_0402_1005Metric, F.Cu at (132.0, 96.8)
- C105, C106, C115, C116, C125, C126, C135, C136, C145, C146, C155, C156, C201, C202, C301, C302: moved to B.Cu
- J1: footprint A_HDJ_Library:PinHeader_1x03_P2.54mm_Vertical -> Connector_PinHeader_2.54mm:PinHeader_1x03_P2.54mm_Vertical
- R87, R88, R89, R90: moved to F.Cu
- moved C481 146.4 mm to (33.0, 213.0)
- moved C482 146.4 mm to (31.5, 213.0)
- moved C483 146.4 mm to (28.5, 210.5)
- moved C484 146.4 mm to (25.5, 215.7)
- moved C485 146.4 mm to (25.5, 211.7)
- moved C486 146.4 mm to (24.0, 211.7)
- moved C487 146.4 mm to (22.7, 211.7)
- moved C488 146.4 mm to (21.5, 211.7)
- moved C489 146.4 mm to (20.0, 211.7)
- moved J481 146.4 mm to (32.2, 218.0)
- moved L481 146.4 mm to (28.0, 207.7)
- moved R481 146.4 mm to (25.5, 214.7)
- moved R482 146.4 mm to (25.5, 213.7)
- moved U480 146.4 mm to (28.5, 212.7)
- moved J82 131.0 mm to (21.8, 185.5)
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Connections:
- net /M.2 M Key/REFCLKM2a+ renamed /M.2 M Key/REFCLKM2+
- net /M.2 M Key/REFCLKM2a- renamed /M.2 M Key/REFCLKM2-
- net /M.2 M Key/REFCLKM2c+ renamed /M.2 M Key/REFCLKM4+
- net /M.2 M Key/REFCLKM2c- renamed /M.2 M Key/REFCLKM4-
- net Net-(C100-Pad1) renamed /PCIe CLK Buffer/RDIF2+
- net Net-(C89-Pad2) renamed /PCIe CLK Buffer/RDIF3-
- net Net-(C90-Pad2) renamed /PCIe CLK Buffer/RDIF3+
- net Net-(C95-Pad1) renamed /PCIe CLK Buffer/RDIF0-
- net Net-(C96-Pad1) renamed /PCIe CLK Buffer/RDIF1-
- net Net-(C97-Pad1) renamed /PCIe CLK Buffer/RDIF2-
- net Net-(C98-Pad1) renamed /PCIe CLK Buffer/RDIF0+
- net Net-(C99-Pad1) renamed /PCIe CLK Buffer/RDIF1+
- net Net-(Q78-DIF0C_LRP) renamed /PCIe CLK Buffer/DIF0-
- net Net-(Q78-DIF0T_LRP) renamed /PCIe CLK Buffer/DIF0+
- net Net-(Q78-DIF1C_LRP) renamed /PCIe CLK Buffer/DIF1-
- net Net-(Q78-DIF1T_LRP) renamed /PCIe CLK Buffer/DIF1+
- net Net-(Q78-DIF2C_LRP) renamed /PCIe CLK Buffer/DIF2-
- net Net-(Q78-DIF2T_LRP) renamed /PCIe CLK Buffer/DIF2+
- net Net-(Q78-DIF3C_LRP) renamed /PCIe CLK Buffer/DIF3-
- net Net-(Q78-DIF3T_LRP) renamed /PCIe CLK Buffer/DIF3+
- C89 pad 1: /M.2 M Key/REFCLKM3+ -> /M.2 M Key/REFCLKM5+
- C90 pad 1: /M.2 M Key/REFCLKM3- -> /M.2 M Key/REFCLKM5-
- C96 pad 2: /M.2 M Key/REFCLKM2b+ -> /M.2 M Key/REFCLKM3+
- C99 pad 2: /M.2 M Key/REFCLKM2b- -> /M.2 M Key/REFCLKM3-
- J100 pad 53: /M.2 M Key/REFCLKM3- -> /LattePanda Module/REFCLK3-
- J100 pad 55: /M.2 M Key/REFCLKM3+ -> /LattePanda Module/REFCLK3+
- J120 pad 52: /M.2 M Key/CLKREQM0 -> /M.2 M Key/CLKREQM2
- J130 pad 52: /M.2 M Key/CLKREQM1 -> /M.2 M Key/CLKREQM3
- J130 pad 53: /M.2 M Key/REFCLKM2b- -> /M.2 M Key/REFCLKM3-
- J130 pad 55: /M.2 M Key/REFCLKM2b+ -> /M.2 M Key/REFCLKM3+
- J140 pad 52: /M.2 M Key/CLKREQM2 -> /M.2 M Key/CLKREQM4
- J150 pad 52: /M.2 M Key/CLKREQM3 -> /M.2 M Key/CLKREQM5
- J150 pad 53: /LattePanda Module/REFCLK3- -> /M.2 M Key/REFCLKM5-
- J150 pad 55: /LattePanda Module/REFCLK3+ -> /M.2 M Key/REFCLKM5+
- Q78 pad 1: /M.2 M Key/CLKREQM0 -> /M.2 M Key/CLKREQM2
- Q78 pad 13: /M.2 M Key/CLKREQM2 -> /M.2 M Key/CLKREQM4
- Q78 pad 16: /M.2 M Key/CLKREQM1 -> /M.2 M Key/CLKREQM3
- Q78 pad 2: unconnected-(Q78-DIF_INC-Pad2) -> /LattePanda Module/REFCLK2+
- Q78 pad 3: unconnected-(Q78-DIF_INT-Pad3) -> /LattePanda Module/REFCLK2-
- Q78 pad 6: /M.2 M Key/CLKREQM3 -> /M.2 M Key/CLKREQM5
Routing:
- net GND: track 149.5 -> 611.3 mm, vias 4 -> 61
- net /LattePanda Module/HSIO_10_RX-: track 10.5 -> 184.6 mm, vias 0 -> 1
- net /LattePanda Module/HSIO_10_RX+: track 10.5 -> 184.6 mm, vias 0 -> 1
- net /M.2 M Key/REFCLKM5+: track 0.00 -> 166.4 mm, vias 0 -> 1
- net /M.2 M Key/REFCLKM5-: track 0.00 -> 166.4 mm, vias 0 -> 1
- net /M.2 M Key/CLKREQM5: track 0.00 -> 164.0 mm, vias 0 -> 1
- net /LattePanda Module/HSIO_10_TX-: track 18.2 -> 176.5 mm
- net /LattePanda Module/HSIO_10_TX+: track 18.2 -> 176.5 mm
- net /LattePanda Module/HSIO_9_RX-: track 9.85 -> 168.1 mm, vias 0 -> 1
- net /LattePanda Module/HSIO_9_RX+: track 9.85 -> 168.1 mm, vias 0 -> 1
- net /LattePanda Module/HSIO_9_TX-: track 18.2 -> 159.8 mm
- net /LattePanda Module/HSIO_9_TX+: track 18.2 -> 159.8 mm
- net /LattePanda Module/HSIO_8_RX+: track 9.85 -> 145.2 mm, vias 0 -> 1
- net /LattePanda Module/HSIO_8_RX-: track 9.85 -> 145.2 mm, vias 0 -> 1
- net /LattePanda Module/REFCLK3+: track 1.97 -> 122.3 mm, vias 0 -> 1
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- added copper zone on In2.Cu, net +12V
- added copper zone on In1.Cu, net GND
Other:
- copper layers 2 -> 4

Commit message: Work
Parts:
- C86, C87, D78, R80, R81, R82, R83, R84, R85, R86, U79: moved to F.Cu
- moved D79 157.9 mm to (173.7, 93.7), turned to 180 degrees
- moved C88 157.8 mm to (167.5, 91.5)
- moved F78 157.2 mm to (167.3, 93.2), turned to 180 degrees
- moved D80 156.7 mm to (171.7, 93.7), turned to 0 degrees
- moved J78 145.5 mm to (166.2, 100.8), turned to 0 degrees
- moved U78 124.6 mm to (84.2, 142.7)
- moved C482 114.8 mm to (132.2, 158.0)
- moved C483 114.8 mm to (129.2, 155.5)
- moved L481 114.8 mm to (128.7, 152.7)
- moved U480 114.8 mm to (129.2, 157.7)
- moved C481 114.8 mm to (133.7, 158.0)
- moved C484 114.8 mm to (126.2, 160.7)
- moved C485 114.8 mm to (126.2, 156.7)
- moved C486 114.8 mm to (124.7, 156.7)
- moved C487 114.8 mm to (123.5, 156.7)
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Routing:
- net /PSU/PWR_EN: track 0.00 -> 660.3 mm, vias 0 -> 7
- net /~{WAKE}: track 0.00 -> 519.8 mm, vias 0 -> 1
- net /~{PLT_RST}: track 0.00 -> 514.7 mm, vias 0 -> 8
- net +3V3: track 15.3 -> 298.7 mm, vias 0 -> 33
- net +5V: track 0.00 -> 218.6 mm, vias 0 -> 22
- net GND: track 611.3 -> 776.9 mm, vias 61 -> 151
- net +12V: track 0.00 -> 156.8 mm, vias 0 -> 129
- net /LattePanda Module/REFCLK1+: track 1.30 -> 126.7 mm, vias 0 -> 2
- net /LattePanda Module/REFCLK1-: track 1.30 -> 126.7 mm, vias 0 -> 2
- net /LattePanda Module/HSIO_11_RX-: track 8.98 -> 133.5 mm
- net /LattePanda Module/HSIO_11_RX+: track 9.44 -> 133.4 mm
- net +3V3 Bios: track 0.00 -> 118.7 mm, vias 0 -> 2
- net /LattePanda Module/HSIO_11_TX-: track 19.8 -> 138.1 mm
- net /LattePanda Module/HSIO_11_TX+: track 20.2 -> 138.1 mm
- net /LattePanda Module/CLKREQ3: track 0.00 -> 115.9 mm, vias 0 -> 3
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- added copper zone on In2.Cu, net +3V3
- added copper zone on In2.Cu, net +3V3a
- added copper zone on In2.Cu, net +3V3cc
- added copper zone on In2.Cu, net +3V3d
- added copper zone on In2.Cu, net +5V
- removed copper zone on B.Cu, net +3V3aa
- removed copper zone on B.Cu, net +3V3b
- removed copper zone on B.Cu, net +3V3bb
- removed copper zone on B.Cu, net +3V3c
- removed copper zone on B.Cu, net +5V
