File: PCB/4 Layer nvme Carrier/BIOS.kicad_sch (KiCad schematic)
At the start: 11 parts, among them U79 W25Q128JVSIQ

Commit message: Silk and BOM changes
Parts:
- C86: LCSC Part # (none) -> C105226; Package (none) -> 0402; Part# (none) -> C105226
- C87: LCSC Part # (none) -> C83056; Package (none) -> 0402; Part# (none) -> C83056
- D78: LCSC Part # (none) -> C239637; Package (none) -> SOD-923; Part# (none) -> C239637
- R80: LCSC Part # (none) -> C93945; Package (none) -> 0402; Part# (none) -> C93945
- R81: LCSC Part # (none) -> C325377; MPN RMC 0402 0R N -> RMC 0402 0R N; Package (none) -> 0402; Part# (none) -> C325377
- R82, R83, R84, R85, R86: LCSC Part # (none) -> C138052; Package (none) -> 0402; Part# (none) -> C138052
- U79: LCSC Part # (none) -> C97521; Package (none) -> SOIC-8-208mil; Part# (none) -> C97521
Changed lines of the file:
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@@
 			)
 		)
-		(property "Part#" ""
+		(property "Part#" "C325377"
 			(at 129.54 93.98 0)
 			(effects
@@
 			)
 		)
-		(property "MPN" " RMC 0402 0R N"
+		(property "MPN" "RMC 0402 0R N"
+			(at 129.54 93.98 0)
+			(effects
+				(font
+					(size 1.27 1.27)
+				)
+				(hide yes)
+			)
+		)
+		(property "Package" "0402"
+			(at 129.54 93.98 0)
+			(effects
+				(font
+					(size 1.27 1.27)
+				)
+				(hide yes)
+			)
+		)
+		(property "LCSC Part #" "C325377"
 			(at 129.54 93.98 0)
 			(effects
@@
 			)
 		)
-		(property "Part#" ""
+		(property "Part#" "C138052"
 			(at 129.54 106.68 0)
 			(effects
@@
 		)
 		(property "MPN" "RC0402FR-0715RL"
+			(at 129.54 106.68 0)
+			(effects
+				(font
+					(size 1.27 1.27)
+				)
+				(hide yes)
+			)
+		)
+		(property "Package" "0402"
+			(at 129.54 106.68 0)
+			(effects
+				(font
+					(size 1.27 1.27)
+				)
+				(hide yes)
+			)
+		)
+		(property "LCSC Part #" "C138052"
 			(at 129.54 106.68 0)
 			(effects
@@
 			)
 		)
-		(property "Part#" ""
+		(property "Part#" "C138052"
 			(at 129.54 113.03 0)
 			(effects
@@
 		)
 		(property "MPN" "RC0402FR-0715RL"
+			(at 129.54 113.03 0)
+			(effects
+				(font
+					(size 1.27 1.27)
+				)
+				(hide yes)
+			)
+		)
+		(property "Package" "0402"
+			(at 129.54 113.03 0)
+			(effects
+				(font
+					(size 1.27 1.27)
+				)
+				(hide yes)
+			)
+		)
+		(property "LCSC Part #" "C138052"
 			(at 129.54 113.03 0)
 			(effects
@@
 			)
 		)
-		(property "Part#" ""
+		(property "Part#" "C138052"
 			(at 129.54 100.33 0)
 			(effects
@@
 		)
 		(property "MPN" "RC0402FR-0715RL"
+			(at 129.54 100.33 0)
+			(effects
+				(font
+					(size 1.27 1.27)
+				)
+				(hide yes)
+			)
+		)
+		(property "Package" "0402"
+			(at 129.54 100.33 0)
+			(effects
+				(font
+					(size 1.27 1.27)
+				)
+				(hide yes)
+			)
+		)
+		(property "LCSC Part #" "C138052"
 			(at 129.54 100.33 0)
 			(effects
@@
 			)
 		)
-		(property "Part#" ""
+		(property "Part#" "C138052"
 			(at 129.54 119.38 0)
 			(effects
@@
 		)
 		(property "MPN" "RC0402FR-0715RL"
+			(at 129.54 119.38 0)
+			(effects
+				(font
+					(size 1.27 1.27)
+				)
+				(hide yes)
+			)
+		)
+		(property "Package" "0402"
+			(at 129.54 119.38 0)
+			(effects
+				(font
+					(size 1.27 1.27)
+				)
+				(hide yes)
+			)
+		)
+		(property "LCSC Part #" "C138052"
 			(at 129.54 119.38 0)
 			(effects
@@
 			)
 		)
-		(property "Part#" ""
+		(property "Part#" "C239637"
 			(at 118.11 74.93 0)
 			(effects
@@
 		)
 		(property "MPN" "RB521C30-2/TR"
+			(at 118.11 74.93 0)
+			(effects
+				(font
+					(size 1.27 1.27)
+				)
+				(hide yes)
+			)
+		)
+		(property "Package" "SOD-923"
+			(at 118.11 74.93 0)
+			(effects
+				(font
+					(size 1.27 1.27)
+				)
+				(hide yes)
+			)
+		)
+		(property "LCSC Part #" "C239637"
 			(at 118.11 74.93 0)
 			(effects
@@
 			)
 		)
-		(property "Part#" ""
+		(property "Part#" "C97521"
 			(at 154.94 101.6 0)
 			(effects
@@
 		)
 		(property "MPN" "W25Q128JVSIQ"
+			(at 154.94 101.6 0)
+			(effects
+				(font
+					(size 1.27 1.27)
+				)
+				(hide yes)
+			)
+		)
+		(property "Package" "SOIC-8-208mil"
+			(at 154.94 101.6 0)
+			(effects
+				(font
+					(size 1.27 1.27)
+				)
+				(hide yes)
+			)
+		)
+		(property "LCSC Part #" "C97521"
 			(at 154.94 101.6 0)
 			(effects
@@
 			)
 		)
-		(property "Part#" ""
+		(property "Part#" "C83056"
 			(at 198.12 102.87 0)
 			(effects
@@
 		)
 		(property "MPN" "0402B104K160CT"
+			(at 198.12 102.87 0)
+			(effects
+				(font
+					(size 1.27 1.27)
+				)
+				(hide yes)
+			)
+		)
+		(property "Package" "0402"
+			(at 198.12 102.87 0)
+			(effects
+				(font
+					(size 1.27 1.27)
+				)
+				(hide yes)
+			)
+		)
+		(property "LCSC Part #" "C83056"
 			(at 198.12 102.87 0)
 			(effects
@@
 			)
 		)
-		(property "Part#" ""
+		(property "Part#" "C105226"
 			(at 180.34 102.87 0)
 			(effects
@@
 		)
 		(property "MPN" "CL05A226MQ5QUNC"
+			(at 180.34 102.87 0)
+			(effects
+				(font
+					(size 1.27 1.27)
+				)
+				(hide yes)
+			)
+		)
+		(property "Package" "0402"
+			(at 180.34 102.87 0)
+			(effects
+				(font
+					(size 1.27 1.27)
+				)
+				(hide yes)
+			)
+		)
+		(property "LCSC Part #" "C105226"
 			(at 180.34 102.87 0)
 			(effects
@@
 			)
 		)
-		(property "Part#" ""
+		(property "Part#" "C93945"
 			(at 129.54 87.63 0)
 			(effects
@@
 		)
 		(property "MPN" "RC0402FR-07120KL"
+			(at 129.54 87.63 0)
+			(effects
+				(font
+					(size 1.27 1.27)
+				)
+				(hide yes)
+			)
+		)
+		(property "Package" "0402"
+			(at 129.54 87.63 0)
+			(effects
+				(font
+					(size 1.27 1.27)
+				)
+				(hide yes)
+			)
+		)
+		(property "LCSC Part #" "C93945"
 			(at 129.54 87.63 0)
 			(effects
@@
 			)
 		)
-		(property "Part#" ""
+		(property "Part#" "C138052"
 			(at 129.54 125.73 0)
 			(effects
@@
 			(at 129.54 125.73 0)
 			(effects
+				(font
+					(size 1.27 1.27)
+				)
+				(hide yes)
+			)
+		)
+		(property "Package" "0402"
+			(at 129.54 125.73 0)
+			(effects
+				(font
+					(size 1.27 1.27)
+				)
+				(hide yes)
+			)
+		)
+		(property "LCSC Part #" "C138052"
+			(at 129.54 125.73 0)
+			(effects
