File: PCB/4 Layer nvme Carrier/HDMI.kicad_sch (KiCad schematic)
At the start: 37 parts, among them J4 HDMI_A, Q1 2N7002, Q2 2SK3018, Q3 2SK3018, Q4 2SK3018, U1 TPAZ1023-04F, U2 TPAZ1023-04F

Commit message: Silk and BOM changes
Parts:
- C17, C18, C19, C20, C21, C22, C23, C24, C25: LCSC Part # (none) -> C77020; Package (none) -> 0402; Part# (none) -> C77020
- D1, D2, D3: LCSC Part # (none) -> C521894; Package (none) -> 0402; Part# (none) -> C521894
- D4: LCSC Part # (none) -> C2828425; Package (none) -> SOD-323; Part# (none) -> C2828425
- F1: LCSC Part # (none) -> C7472536; Package (none) -> 0603; Part# (none) -> C7472536
- J4: LCSC Part # (none) -> C2858275; Package (none) -> Plugin; Part# (none) -> C916313
- Q1: LCSC Part # (none) -> C7603342; Package (none) -> SOT-23; Part# (none) -> C7603342
- Q2, Q3, Q4: LCSC Part # (none) -> C475593; Package (none) -> SOT-23; Part# (none) -> C475593
- R10, R13, R14, R16, R17, R7, R8, R9: LCSC Part # (none) -> C114877; Package (none) -> 0402; Part# (none) -> C114877
- R11: LCSC Part # (none) -> C106235; Package (none) -> 0402; Part# (none) -> C106235
- R15, R18, R19, R3, R5: LCSC Part # (none) -> C114762; Package (none) -> 0402; Part# (none) -> C114762
- R4: LCSC Part # (none) -> C138033; Package (none) -> 0402; Part# (none) -> C138033
- R6: LCSC Part # (none) -> C185442; Package (none) -> 0402; Part# (none) -> C185442
- U1, U2: LCSC Part # (none) -> C2827676; Package (none) -> DFN2510; Part# (none) -> C2827676
