File: PCB/4 Layer nvme Carrier/LattePanda Module.kicad_sch (KiCad schematic)
At the start: 13 parts, among them J1 Conn_01x03_Pin, J11 Conn_01x03_Pin

Commit message: Prototyp_1
Parts:
- J1: MPN 2.54-1*3 -> PZ2.54-1*3; now not fitted
- J11: MPN (none) -> PZ2.54-1*3; now not fitted
- R78, R79: value 10K/1% -> 100K/1%; footprint Resistor_SMD:R_0402_1005Metric -> A_HDJ_Library:R_0402_1005Metric; MPN (none) -> RC0402FR-07100KL; now fitted
Connections:
- net TSENSE: now reaches A1.9 (TSENSE)
- no-connect marks 95 -> 94
Changed lines of the file:
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@@
 	)
 	(no_connect
-		(at 351.79 60.96)
-	)
-	(no_connect
 		(at 351.79 195.58)
 	)
@@
 	(wire
 		(pts
+			(xy 351.79 60.96) (xy 369.57 60.96)
+		)
+		(stroke
+			(width 0)
+			(type default)
+		)
+	)
+	(wire
+		(pts
 			(xy 238.76 175.26) (xy 270.51 175.26)
 		)
@@
 		)
 	)
+	(hierarchical_label "TSENSE"
+		(shape input)
+		(at 369.57 60.96 0)
+		(fields_autoplaced yes)
+		(effects
+			(font
+				(size 1.27 1.27)
+			)
+			(justify left)
+		)
+	)
 	(hierarchical_label "HSIO_6_RX+"
 		(shape input)
@@
 		(in_bom yes)
 		(on_board yes)
-		(dnp no)
+		(dnp yes)
 		(fields_autoplaced yes)
 		(property "Reference" "J1"
@@
 			)
 		)
-		(property "MPN" "2.54-1*3"
+		(property "MPN" "PZ2.54-1*3"
 			(at 215.9 63.5 90)
 			(effects
@@
 		(in_bom yes)
 		(on_board yes)
-		(dnp yes)
+		(dnp no)
 		(fields_autoplaced yes)
 		(property "Reference" "R79"
@@
 			)
 		)
-		(property "Value" "10K/1%"
+		(property "Value" "100K/1%"
 			(at 396.24 121.9199 0)
 			(effects
@@
 			)
 		)
-		(property "Footprint" "Resistor_SMD:R_0402_1005Metric"
+		(property "Footprint" "A_HDJ_Library:R_0402_1005Metric"
 			(at 391.922 120.65 90)
 			(effects
@@
 			)
 		)
-		(property "Datasheet" "~"
+		(property "Datasheet" "https://wmsc.lcsc.com/wmsc/upload/file/pdf/v2/lcsc/2304140030_YAGEO-RC0402FR-07100KL_C60491.pdf"
 			(at 393.7 120.65 0)
 			(effects
@@
 			)
 		)
+		(property "MPN" "RC0402FR-07100KL"
+			(at 393.7 120.65 0)
+			(effects
+				(font
+					(size 1.27 1.27)
+				)
+				(hide yes)
+			)
+		)
 		(pin "2"
 		)
@@
 		(in_bom yes)
 		(on_board yes)
-		(dnp yes)
+		(dnp no)
 		(fields_autoplaced yes)
 		(property "Reference" "R78"
@@
 			)
 		)
-		(property "Value" "10K/1%"
+		(property "Value" "100K/1%"
 			(at 383.54 121.9199 0)
 			(effects
@@
 			)
 		)
-		(property "Footprint" "Resistor_SMD:R_0402_1005Metric"
+		(property "Footprint" "A_HDJ_Library:R_0402_1005Metric"
 			(at 379.222 120.65 90)
 			(effects
@@
 			)
 		)
-		(property "Datasheet" "~"
+		(property "Datasheet" "https://wmsc.lcsc.com/wmsc/upload/file/pdf/v2/lcsc/2304140030_YAGEO-RC0402FR-07100KL_C60491.pdf"
 			(at 381 120.65 0)
 			(effects
@@
 			)
 		)
+		(property "MPN" "RC0402FR-07100KL"
+			(at 381 120.65 0)
+			(effects
+				(font
+					(size 1.27 1.27)
+				)
+				(hide yes)
+			)
+		)
 		(pin "2"
 		)
@@
 		(in_bom yes)
 		(on_board yes)
-		(dnp no)
+		(dnp yes)
 		(fields_autoplaced yes)
 		(property "Reference" "J11"
@@
 			(at 379.73 271.78 0)
 			(effects
+				(font
+					(size 1.27 1.27)
+				)
+				(hide yes)
+			)
+		)
+		(property "MPN" "PZ2.54-1*3"
+			(at 379.73 271.78 0)
+			(effects

Commit message: Silk and BOM changes
Parts:
- A1: LCSC Part # (none) -> C962126; Package (none) -> SMD,P=0.5mm,Surface Mount，Right Angle; Part# (none) -> C962126
- BT1: LCSC Part # (none) -> C70381; MPN S8411-45R -> CR1220-2; MPN_alt (none) -> S8411-45R; Package (none) -> SMD; Part# (none) -> C70381
- H5, H6: Package (none) -> MountingHole; now left out of the parts list
- J1, J11: Package (none) -> Jumper; now fitted
- R1: LCSC Part # (none) -> C106235; Package (none) -> 0402; Part# (none) -> C106235
- R2, R95: LCSC Part # (none) -> C60490; Package (none) -> 0402; Part# (none) -> C60490
- R76, R77, R78, R79: LCSC Part # (none) -> C60491; Package (none) -> 0402; Part# (none) -> C60491
