File: PCB/4 Layer nvme Carrier/PCIe CLK Buffer.kicad_sch (KiCad schematic)
At the start: 23 parts

Commit message: Prototyp_1
Parts:
- Q78: value ~ -> 9DBL411BGLFT
- R96, R97, R98, R99: value 10K/1% -> 100K/1%; footprint Resistor_SMD:R_0402_1005Metric -> A_HDJ_Library:R_0402_1005Metric; MPN (none) -> RC0402FR-07100KL; now fitted
Connections:
- net REFCLKB0+: now also C98.2; no longer C95.2
- net REFCLKB0-: now also C95.2; no longer C98.2
- net REFCLKB1+: now also C99.2; no longer C96.2
- net REFCLKB1-: now also C96.2; no longer C99.2
- net REFCLKB2+: now also C100.2; no longer C97.2
- net REFCLKB2-: now also C97.2; no longer C100.2
- net REFCLKB3+: now also C90.1; no longer C89.1
- net REFCLKB3-: now also C89.1; no longer C90.1
Changed lines of the file:
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@@
 	(wire
 		(pts
+			(xy 223.52 93.98) (xy 227.33 93.98)
+		)
+		(stroke
+			(width 0)
+			(type default)
+		)
+	)
+	(wire
+		(pts
 			(xy 163.83 86.36) (xy 163.83 59.69)
 		)
@@
 	(wire
 		(pts
+			(xy 215.9 107.95) (xy 227.33 107.95)
+		)
+		(stroke
+			(width 0)
+			(type default)
+		)
+	)
+	(wire
+		(pts
 			(xy 128.27 104.14) (xy 130.81 104.14)
 		)
@@
 	(wire
 		(pts
-			(xy 215.9 91.44) (xy 227.33 91.44)
-		)
-		(stroke
-			(width 0)
-			(type default)
-		)
-	)
-	(wire
-		(pts
 			(xy 176.53 110.49) (xy 176.53 104.14)
 		)
@@
 	(wire
 		(pts
-			(xy 215.9 107.95) (xy 227.33 107.95)
+			(xy 80.01 99.06) (xy 90.17 99.06)
 		)
 		(stroke
@@
 	(wire
 		(pts
-			(xy 80.01 99.06) (xy 90.17 99.06)
+			(xy 223.52 110.49) (xy 227.33 110.49)
 		)
 		(stroke
@@
 	(wire
 		(pts
-			(xy 223.52 93.98) (xy 227.33 93.98)
+			(xy 215.9 91.44) (xy 227.33 91.44)
 		)
 		(stroke
@@
 	(wire
 		(pts
-			(xy 223.52 110.49) (xy 227.33 110.49)
-		)
-		(stroke
-			(width 0)
-			(type default)
-		)
-	)
-	(wire
-		(pts
 			(xy 177.8 93.98) (xy 179.07 93.98)
 		)
@@
 		)
 	)
-	(hierarchical_label "REFCLKB3-"
+	(hierarchical_label "REFCLKB3+"
 		(shape output)
 		(at 80.01 99.06 180)
@@
 		)
 	)
-	(hierarchical_label "REFCLKB0-"
+	(hierarchical_label "REFCLKB0+"
 		(shape output)
 		(at 227.33 77.47 0)
@@
 		)
 	)
-	(hierarchical_label "REFCLKB1-"
+	(hierarchical_label "REFCLKB1+"
 		(shape output)
 		(at 227.33 93.98 0)
@@
 		)
 	)
-	(hierarchical_label "REFCLKB3+"
+	(hierarchical_label "REFCLKB3-"
 		(shape output)
 		(at 80.01 96.52 180)
@@
 		)
 	)
-	(hierarchical_label "REFCLKB1+"
+	(hierarchical_label "REFCLKB1-"
 		(shape output)
 		(at 227.33 91.44 0)
@@
 		)
 	)
-	(hierarchical_label "REFCLKB0+"
+	(hierarchical_label "REFCLKB0-"
 		(shape output)
 		(at 227.33 74.93 0)
@@
 	(hierarchical_label "REFCLKB2-"
 		(shape output)
-		(at 227.33 110.49 0)
+		(at 227.33 107.95 0)
 		(fields_autoplaced yes)
 		(effects
@@
 	(hierarchical_label "REFCLKB2+"
 		(shape output)
-		(at 227.33 107.95 0)
+		(at 227.33 110.49 0)
 		(fields_autoplaced yes)
 		(effects
@@
 		(in_bom yes)
 		(on_board yes)
-		(dnp yes)
+		(dnp no)
 		(fields_autoplaced yes)
 		(property "Reference" "R96"
@@
 			)
 		)
-		(property "Value" "10K/1%"
+		(property "Value" "100K/1%"
 			(at 252.73 105.4099 0)
 			(effects
@@
 			)
 		)
-		(property "Footprint" "Resistor_SMD:R_0402_1005Metric"
+		(property "Footprint" "A_HDJ_Library:R_0402_1005Metric"
 			(at 248.412 104.14 90)
 			(effects
@@
 			)
 		)
-		(property "Datasheet" "~"
+		(property "Datasheet" "https://wmsc.lcsc.com/wmsc/upload/file/pdf/v2/lcsc/2304140030_YAGEO-RC0402FR-07100KL_C60491.pdf"
 			(at 250.19 104.14 0)
 			(effects
@@
 			)
 		)
+		(property "MPN" "RC0402FR-07100KL"
+			(at 250.19 104.14 0)
+			(effects
+				(font
+					(size 1.27 1.27)
+				)
+				(hide yes)
+			)
+		)
 		(pin "2"
 		)
@@
 		(in_bom yes)
 		(on_board yes)
-		(dnp yes)
+		(dnp no)
 		(fields_autoplaced yes)
 		(property "Reference" "R99"
@@
 			)
 		)
-		(property "Value" "10K/1%"
+		(property "Value" "100K/1%"
 			(at 53.34 77.4699 0)
 			(effects
@@
 			)
 		)
-		(property "Footprint" "Resistor_SMD:R_0402_1005Metric"
+		(property "Footprint" "A_HDJ_Library:R_0402_1005Metric"
 			(at 49.022 76.2 90)
 			(effects
@@
 			)
 		)
-		(property "Datasheet" "~"
+		(property "Datasheet" "https://wmsc.lcsc.com/wmsc/upload/file/pdf/v2/lcsc/2304140030_YAGEO-RC0402FR-07100KL_C60491.pdf"
 			(at 50.8 76.2 0)
 			(effects
@@
 			)
 		)
+		(property "MPN" "RC0402FR-07100KL"
+			(at 50.8 76.2 0)
+			(effects
+				(font
+					(size 1.27 1.27)
+				)
+				(hide yes)
+			)
+		)
 		(pin "2"
 		)
@@
 		(in_bom yes)
 		(on_board yes)
-		(dnp yes)
+		(dnp no)
 		(fields_autoplaced yes)
 		(property "Reference" "R98"
@@
 			)
 		)
-		(property "Value" "10K/1%"
+		(property "Value" "100K/1%"
 			(at 53.34 95.2499 0)
 			(effects
@@
 			)
 		)
-		(property "Footprint" "Resistor_SMD:R_0402_1005Metric"
+		(property "Footprint" "A_HDJ_Library:R_0402_1005Metric"
 			(at 49.022 93.98 90)
 			(effects
@@
 			)
 		)
-		(property "Datasheet" "~"
+		(property "Datasheet" "https://wmsc.lcsc.com/wmsc/upload/file/pdf/v2/lcsc/2304140030_YAGEO-RC0402FR-07100KL_C60491.pdf"
 			(at 50.8 93.98 0)
 			(effects
@@
 			)
 		)
+		(property "MPN" "RC0402FR-07100KL"
+			(at 50.8 93.98 0)
+			(effects
+				(font
+					(size 1.27 1.27)
+				)
+				(hide yes)
+			)
+		)
 		(pin "2"
 		)
@@
 		(in_bom yes)
 		(on_board yes)
-		(dnp yes)
+		(dnp no)
 		(fields_autoplaced yes)
 		(property "Reference" "R97"
@@
 			)
 		)
-		(property "Value" "10K/1%"
+		(property "Value" "100K/1%"
 			(at 252.73 87.6299 0)
 			(effects
@@
 			)
 		)
-		(property "Footprint" "Resistor_SMD:R_0402_1005Metric"
+		(property "Footprint" "A_HDJ_Library:R_0402_1005Metric"
 			(at 248.412 86.36 90)
 			(effects
@@
 			)
 		)
-		(property "Datasheet" "~"
+		(property "Datasheet" "https://wmsc.lcsc.com/wmsc/upload/file/pdf/v2/lcsc/2304140030_YAGEO-RC0402FR-07100KL_C60491.pdf"
 			(at 250.19 86.36 0)
 			(effects
@@
 			)
 		)
+		(property "MPN" "RC0402FR-07100KL"
+			(at 250.19 86.36 0)
+			(effects
+				(font
+					(size 1.27 1.27)
+				)
+				(hide yes)
+			)
+		)
 		(pin "2"
 		)
@@
 			)
 		)
-		(property "Value" "~"
+		(property "Value" "9DBL411BGLFT"
 			(at 144.78 77.47 0)
 			(effects

Commit message: wrong Partnumber for the 33R
Parts:
- R87, R88, R89, R90, R91, R92, R93, R94: MPN RC0402FR-071KL -> RC0402JR-0733RP
Changed lines of the file:
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@@
 			)
 		)
-		(property "MPN" "RC0402FR-071KL"
+		(property "MPN" "RC0402JR-0733RP"
 			(at 182.88 110.49 0)
 			(effects
@@
 			)
 		)
-		(property "MPN" "RC0402FR-071KL"
+		(property "MPN" "RC0402JR-0733RP"
 			(at 182.88 91.44 0)
 			(effects
@@
 			)
 		)
-		(property "MPN" "RC0402FR-071KL"
+		(property "MPN" "RC0402JR-0733RP"
 			(at 182.88 107.95 0)
 			(effects
@@
 			)
 		)
-		(property "MPN" "RC0402FR-071KL"
+		(property "MPN" "RC0402JR-0733RP"
 			(at 182.88 93.98 0)
 			(effects
@@
 			)
 		)
-		(property "MPN" "RC0402FR-071KL"
+		(property "MPN" "RC0402JR-0733RP"
 			(at 116.84 99.06 0)
 			(effects
@@
 			)
 		)
-		(property "MPN" "RC0402FR-071KL"
+		(property "MPN" "RC0402JR-0733RP"
 			(at 182.88 77.47 0)
 			(effects
@@
 			)
 		)
-		(property "MPN" "RC0402FR-071KL"
+		(property "MPN" "RC0402JR-0733RP"
 			(at 182.88 74.93 0)
 			(effects
@@
 			)
 		)
-		(property "MPN" "RC0402FR-071KL"
+		(property "MPN" "RC0402JR-0733RP"
 			(at 116.84 96.52 0)
 			(effects

Commit message: Silk and BOM changes
Parts:
- C100, C89, C90, C94, C95, C96, C97, C98, C99: LCSC Part # (none) -> C83056; Package (none) -> 0402; Part# (none) -> C83056
- C93: LCSC Part # (none) -> C105226; Package (none) -> 0402; Part# (none) -> C105226
- Q78: LCSC Part # (none) -> C2649348; Package (none) -> TSSOP-20; Part# (none) -> C2649348
- R87, R88, R89, R90, R91, R92, R93, R94: LCSC Part # (none) -> C851857; Package (none) -> 0402; Part# (none) -> C851857
- R96, R97, R98, R99: LCSC Part # (none) -> C60491; Package (none) -> 0402; Part# (none) -> C60491
