File: PCB/4 Layer nvme Carrier/USB.kicad_sch (KiCad schematic)
At the start: 18 parts, among them J2 USB_A_Stacked, J3 USB3_A, J78 USB_A, U3 ULC0524P, U4 ULC0524P

Commit message: Silk and BOM changes
Parts:
- C28, C29: LCSC Part # (none) -> C77020; Package (none) -> 0402; Part# (none) -> C77020
- C30, C32, C88: LCSC Part # (none) -> C86295; Package (none) -> 0603; Part# (none) -> C86295
- D5, D6, D79, D80: LCSC Part # (none) -> C521894; Package (none) -> 0402; Part# (none) -> C521894
- F2, F3, F78: LCSC Part # (none) -> C883112; Package (none) -> 0805; Part# (none) -> C883112
- F5: LCSC Part # (none) -> C2757931; Package (none) -> 0805; Part# (none) -> C2757931
- J2: LCSC Part # (none) -> C456021; MPN UJ2-ADH-W1-TH -> UJ2-ADH-1-TH; MPN_alt (none) -> AF SS-JB17.6; Package (none) -> Plugin; Part# (none) -> C3197848
- J3: MPN_alt (none) -> 692122030100; Package (none) -> Plugin; now left out of the parts list
- J78: LCSC Part # (none) -> C586225; Package (none) -> Plugin; Part# (none) -> C586225
- U3, U4: LCSC Part # (none) -> C2835428; Package (none) -> DFN2510; Part# (none) -> C2835428

Commit message: USB 3 listed in BOM
Parts:
- J3: now in the parts list
Changed lines of the file:
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@@
 		(unit 1)
 		(exclude_from_sim no)
-		(in_bom no)
+		(in_bom yes)
 		(on_board yes)
 		(dnp no)
