File: PCB/4 Layer nvme Carrier/PCIe.kicad_sch (KiCad schematic)
At the start: 22 parts, among them J200 Bus_PCI_Express_x4, J300 Bus_PCI_Express_x4

Commit message: Silk and BOM changes
Parts:
- C201, C202, C301, C302: LCSC Part # (none) -> C5159775; Package (none) -> 0402; Part# (none) -> C5159775
- C203, C204, C207, C209, C303, C304, C307, C309: LCSC Part # (none) -> C77020; Package (none) -> 0402; Part# (none) -> C77020
- C205, C206, C305, C306: LCSC Part # (none) -> C2886300; MPN PM101M025E077PTR -> VT1E101M-CRE54; MPN_alt (none) -> PM101M025E077PTR; Package (none) -> SMD,D6.3xL7.7mm; Part# (none) -> C2886300
- C208, C308: LCSC Part # (none) -> C315248; Package (none) -> 0402; Part# (none) -> C315248
- C210, C310: LCSC Part # (none) -> C384654; Package (none) -> SMD,D6.3xL7.7mm; Part# (none) -> C384654
- J200, J300: LCSC Part # (none) -> C2926855; Package (none) -> Plugin,P=2mm; Part# (none) -> C2926855

Commit message: new JPG, new 3V3 names and del the M.2 60mm mounts
Connections:
- net +3V3d renamed +3V3g
Changed lines of the file:
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@@
 			)
 		)
-		(property "Value" "+3V3d"
+		(property "Value" "+3V3g"
 			(at 393.7 153.162 0)
 			(effects
