File: PCB/4 Layer nvme Carrier/M.2 M Key.kicad_sch (KiCad schematic)
At the start: 78 parts, among them J100 Bus_M.2_Socket_M, J110 Bus_M.2_Socket_M, J120 Bus_M.2_Socket_M, J130 Bus_M.2_Socket_M, J140 Bus_M.2_Socket_M, J150 Bus_M.2_Socket_M

Commit message: Prototyp_1
Parts:
- H1032, H1042, H1060, H1080, H1130, H1142, H1160, H1180, H1230, H1242, H1260, H1280, H1330, H1342, H1360, H1380, H1430, H1442, H1460, H1480, H1530, H1542, H1560, H1580: now left out of the parts list
Changed lines of the file:
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@@
 		(unit 1)
 		(exclude_from_sim no)
-		(in_bom yes)
+		(in_bom no)
 		(on_board yes)
 		(dnp no)
@@
 		(unit 1)
 		(exclude_from_sim no)
-		(in_bom yes)
+		(in_bom no)
 		(on_board yes)
 		(dnp no)
@@
 		(unit 1)
 		(exclude_from_sim no)
-		(in_bom yes)
+		(in_bom no)
 		(on_board yes)
 		(dnp no)
@@
 		(unit 1)
 		(exclude_from_sim no)
-		(in_bom yes)
+		(in_bom no)
 		(on_board yes)
 		(dnp no)
@@
 		(unit 1)
 		(exclude_from_sim no)
-		(in_bom yes)
+		(in_bom no)
 		(on_board yes)
 		(dnp no)
@@
 		(unit 1)
 		(exclude_from_sim no)
-		(in_bom yes)
+		(in_bom no)
 		(on_board yes)
 		(dnp no)
@@
 		(unit 1)
 		(exclude_from_sim no)
-		(in_bom yes)
+		(in_bom no)
 		(on_board yes)
 		(dnp no)
@@
 		(unit 1)
 		(exclude_from_sim no)
-		(in_bom yes)
+		(in_bom no)
 		(on_board yes)
 		(dnp no)
@@
 		(unit 1)
 		(exclude_from_sim no)
-		(in_bom yes)
+		(in_bom no)
 		(on_board yes)
 		(dnp no)
@@
 		(unit 1)
 		(exclude_from_sim no)
-		(in_bom yes)
+		(in_bom no)
 		(on_board yes)
 		(dnp no)
@@
 		(unit 1)
 		(exclude_from_sim no)
-		(in_bom yes)
+		(in_bom no)
 		(on_board yes)
 		(dnp no)
@@
 		(unit 1)
 		(exclude_from_sim no)
-		(in_bom yes)
+		(in_bom no)
 		(on_board yes)
 		(dnp no)
@@
 		(unit 1)
 		(exclude_from_sim no)
-		(in_bom yes)
+		(in_bom no)
 		(on_board yes)
 		(dnp no)
@@
 		(unit 1)
 		(exclude_from_sim no)
-		(in_bom yes)
+		(in_bom no)
 		(on_board yes)
 		(dnp no)
@@
 		(unit 1)
 		(exclude_from_sim no)
-		(in_bom yes)
+		(in_bom no)
 		(on_board yes)
 		(dnp no)
@@
 		(unit 1)
 		(exclude_from_sim no)
-		(in_bom yes)
+		(in_bom no)
 		(on_board yes)
 		(dnp no)
@@
 		(unit 1)
 		(exclude_from_sim no)
-		(in_bom yes)
+		(in_bom no)
 		(on_board yes)
 		(dnp no)
@@
 		(unit 1)
 		(exclude_from_sim no)
-		(in_bom yes)
+		(in_bom no)
 		(on_board yes)
 		(dnp no)
@@
 		(unit 1)
 		(exclude_from_sim no)
-		(in_bom yes)
+		(in_bom no)
 		(on_board yes)
 		(dnp no)
@@
 		(unit 1)
 		(exclude_from_sim no)
-		(in_bom yes)
+		(in_bom no)
 		(on_board yes)
 		(dnp no)
@@
 		(unit 1)
 		(exclude_from_sim no)
-		(in_bom yes)
+		(in_bom no)
 		(on_board yes)
 		(dnp no)
@@
 		(unit 1)
 		(exclude_from_sim no)
-		(in_bom yes)
+		(in_bom no)
 		(on_board yes)
 		(dnp no)
@@
 		(unit 1)
 		(exclude_from_sim no)
-		(in_bom yes)
+		(in_bom no)
 		(on_board yes)
 		(dnp no)
@@
 		(unit 1)
 		(exclude_from_sim no)
-		(in_bom yes)
+		(in_bom no)
 		(on_board yes)
 		(dnp no)
@@
 		(unit 1)
 		(exclude_from_sim no)
-		(in_bom yes)
+		(in_bom no)
 		(on_board yes)
 		(dnp no)
@@
 		(unit 1)
 		(exclude_from_sim no)
-		(in_bom yes)
+		(in_bom no)
 		(on_board yes)
 		(dnp no)
@@
 		(unit 1)
 		(exclude_from_sim no)
-		(in_bom yes)
+		(in_bom no)
 		(on_board yes)
 		(dnp no)
@@
 		(unit 1)
 		(exclude_from_sim no)
-		(in_bom yes)
+		(in_bom no)
 		(on_board yes)
 		(dnp no)
@@
 		(unit 1)
 		(exclude_from_sim no)
-		(in_bom yes)
+		(in_bom no)
 		(on_board yes)
 		(dnp no)
@@
 		(unit 1)
 		(exclude_from_sim no)
-		(in_bom yes)
+		(in_bom no)
 		(on_board yes)
 		(dnp no)
@@
 		(unit 1)
 		(exclude_from_sim no)
-		(in_bom yes)
+		(in_bom no)
 		(on_board yes)
 		(dnp no)
@@
 		(unit 1)
 		(exclude_from_sim no)
-		(in_bom yes)
+		(in_bom no)
 		(on_board yes)
 		(dnp no)
@@
 		(unit 1)
 		(exclude_from_sim no)
-		(in_bom yes)
+		(in_bom no)
 		(on_board yes)
 		(dnp no)
@@
 		(unit 1)
 		(exclude_from_sim no)
-		(in_bom yes)
+		(in_bom no)
 		(on_board yes)
 		(dnp no)
@@
 		(unit 1)
 		(exclude_from_sim no)
-		(in_bom yes)
+		(in_bom no)
 		(on_board yes)
 		(dnp no)
@@
 		(unit 1)
 		(exclude_from_sim no)
-		(in_bom yes)
+		(in_bom no)
 		(on_board yes)
 		(dnp no)
@@
 		(unit 1)
 		(exclude_from_sim no)
-		(in_bom yes)
+		(in_bom no)
 		(on_board yes)
 		(dnp no)
@@
 		(unit 1)
 		(exclude_from_sim no)
-		(in_bom yes)
+		(in_bom no)
 		(on_board yes)
 		(dnp no)
@@
 		(unit 1)
 		(exclude_from_sim no)
-		(in_bom yes)
+		(in_bom no)
 		(on_board yes)
 		(dnp no)
@@
 		(unit 1)
 		(exclude_from_sim no)
-		(in_bom yes)
+		(in_bom no)
 		(on_board yes)
 		(dnp no)
@@
 		(unit 1)
 		(exclude_from_sim no)
-		(in_bom yes)
+		(in_bom no)
 		(on_board yes)
 		(dnp no)
@@
 		(unit 1)
 		(exclude_from_sim no)
-		(in_bom yes)
+		(in_bom no)
 		(on_board yes)
 		(dnp no)
@@
 		(unit 1)
 		(exclude_from_sim no)
-		(in_bom yes)
+		(in_bom no)
 		(on_board yes)
 		(dnp no)
@@
 		(unit 1)
 		(exclude_from_sim no)
-		(in_bom yes)
+		(in_bom no)
 		(on_board yes)
 		(dnp no)
@@
 		(unit 1)
 		(exclude_from_sim no)
-		(in_bom yes)
+		(in_bom no)
 		(on_board yes)
 		(dnp no)
@@
 		(unit 1)
 		(exclude_from_sim no)
-		(in_bom yes)
+		(in_bom no)
 		(on_board yes)
 		(dnp no)
@@
 		(unit 1)
 		(exclude_from_sim no)
-		(in_bom yes)
+		(in_bom no)
 		(on_board yes)
 		(dnp no)
@@
 		(unit 1)
 		(exclude_from_sim no)
-		(in_bom yes)
+		(in_bom no)
 		(on_board yes)
 		(dnp no)

Commit message: Silk and BOM changes
Parts:
- C101, C103, C111, C113, C121, C123, C131, C133, C141, C143, C151, C153: LCSC Part # (none) -> C315248; Package (none) -> 0402; Part# (none) -> C315248
- C102, C104, C112, C114, C122, C124, C132, C134, C142, C144, C152, C154: LCSC Part # (none) -> C77020; Package (none) -> 0402; Part# (none) -> C77020
- C105, C106, C115, C116, C125, C126, C135, C136, C145, C146, C155, C156: LCSC Part # (none) -> C5159775; Package (none) -> 0402; Part# (none) -> C5159775
- D101, D111, D121, D131, D141, D151: LCSC Part # (none) -> C434423; Package (none) -> 0603; Part# (none) -> C434423
- H1032, H1042, H1060, H1080, H1130, H1142, H1160, H1180, H1230, H1242, H1260, H1280, H1330, H1342, H1360, H1380, H1430, H1442, H1460, H1480, H1530, H1542, H1560, H1580: Package (none) -> MountingHole
- J100, J110, J120, J130, J140, J150: LCSC Part # (none) -> C590854; MPN_alt (none) -> APCI0079-P002A; Package (none) -> SMD,P=0.5mm,Surface Mount，Right Angle; Part# (none) -> C590854
- R102, R112, R122, R132, R142, R152: LCSC Part # (none) -> C114762; Package (none) -> 0402; Part# (none) -> C114762

Commit message: new JPG, new 3V3 names and del the M.2 60mm mounts
Parts:
- H1060, H1160, H1260, H1360, H1460, H1560: now not fitted
Connections:
- net +3V3aa: no longer C131.2, C132.2, C133.2, C134.2, J130.12 (3.3V), J130.14 (3.3V), J130.16 (3.3V), J130.18 (3.3V), J130.2 (3.3V), J130.4 (3.3V), J130.70 (3.3V), J130.72 (3.3V), J130.74 (3.3V)
- net +3V3bb: no longer C141.2, C142.2, C143.2, C144.2, J140.12 (3.3V), J140.14 (3.3V), J140.16 (3.3V), J140.18 (3.3V), J140.2 (3.3V), J140.4 (3.3V), J140.70 (3.3V), J140.72 (3.3V), J140.74 (3.3V)
- net +3V3cc: no longer C151.2, C152.2, C153.2, C154.2, J150.12 (3.3V), J150.14 (3.3V), J150.16 (3.3V), J150.18 (3.3V), J150.2 (3.3V), J150.4 (3.3V), J150.70 (3.3V), J150.72 (3.3V), J150.74 (3.3V)
- new net +3V3d: C131.2, C132.2, C133.2, C134.2, J130.12 (3.3V), J130.14 (3.3V), J130.16 (3.3V), J130.18 (3.3V), J130.2 (3.3V), J130.4 (3.3V), J130.70 (3.3V), J130.72 (3.3V), J130.74 (3.3V)
- new net +3V3e: C141.2, C142.2, C143.2, C144.2, J140.12 (3.3V), J140.14 (3.3V), J140.16 (3.3V), J140.18 (3.3V), J140.2 (3.3V), J140.4 (3.3V), J140.70 (3.3V), J140.72 (3.3V), J140.74 (3.3V)
- new net +3V3f: C151.2, C152.2, C153.2, C154.2, J150.12 (3.3V), J150.14 (3.3V), J150.16 (3.3V), J150.18 (3.3V), J150.2 (3.3V), J150.4 (3.3V), J150.70 (3.3V), J150.72 (3.3V), J150.74 (3.3V)
Changed lines of the file:
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@@
 			)
 		)
-		(property "Value" "+3V3cc"
+		(property "Value" "+3V3f"
 			(at 482.6 212.598 0)
 			(effects
@@
 		(exclude_from_sim no)
 		(in_bom no)
-		(on_board yes)
-		(dnp no)
+		(on_board no)
+		(dnp yes)
 		(fields_autoplaced yes)
 		(property "Reference" "#PWR0157"
@@
 		(exclude_from_sim no)
 		(in_bom no)
-		(on_board yes)
-		(dnp no)
+		(on_board no)
+		(dnp yes)
 		(fields_autoplaced yes)
 		(property "Reference" "#PWR0165"
@@
 		(exclude_from_sim no)
 		(in_bom no)
-		(on_board yes)
-		(dnp no)
+		(on_board no)
+		(dnp yes)
 		(fields_autoplaced yes)
 		(property "Reference" "H1560"
@@
 		(exclude_from_sim no)
 		(in_bom no)
-		(on_board yes)
-		(dnp no)
+		(on_board no)
+		(dnp yes)
 		(fields_autoplaced yes)
 		(property "Reference" "#PWR0177"
@@
 		(exclude_from_sim no)
 		(in_bom no)
-		(on_board yes)
-		(dnp no)
+		(on_board no)
+		(dnp yes)
 		(fields_autoplaced yes)
 		(property "Reference" "#PWR0161"
@@
 		(exclude_from_sim no)
 		(in_bom no)
-		(on_board yes)
-		(dnp no)
+		(on_board no)
+		(dnp yes)
 		(fields_autoplaced yes)
 		(property "Reference" "H1360"
@@
 		(exclude_from_sim no)
 		(in_bom no)
-		(on_board yes)
-		(dnp no)
+		(on_board no)
+		(dnp yes)
 		(fields_autoplaced yes)
 		(property "Reference" "#PWR0173"
@@
 			)
 		)
-		(property "Value" "+3V3aa"
+		(property "Value" "+3V3d"
 			(at 121.92 208.026 0)
 			(effects
@@
 		(exclude_from_sim no)
 		(in_bom no)
-		(on_board yes)
-		(dnp no)
+		(on_board no)
+		(dnp yes)
 		(fields_autoplaced yes)
 		(property "Reference" "H1060"
@@
 		(exclude_from_sim no)
 		(in_bom no)
-		(on_board yes)
-		(dnp no)
+		(on_board no)
+		(dnp yes)
 		(fields_autoplaced yes)
 		(property "Reference" "H1460"
@@
 			)
 		)
-		(property "Value" "+3V3bb"
+		(property "Value" "+3V3e"
 			(at 293.37 211.836 0)
 			(effects
@@
 		(exclude_from_sim no)
 		(in_bom no)
-		(on_board yes)
-		(dnp no)
+		(on_board no)
+		(dnp yes)
 		(fields_autoplaced yes)
 		(property "Reference" "H1160"
@@
 		(exclude_from_sim no)
 		(in_bom no)
-		(on_board yes)
-		(dnp no)
+		(on_board no)
+		(dnp yes)
 		(fields_autoplaced yes)
 		(property "Reference" "H1260"
@@
 		(exclude_from_sim no)
 		(in_bom no)
-		(on_board yes)
-		(dnp no)
+		(on_board no)
+		(dnp yes)
 		(fields_autoplaced yes)
 		(property "Reference" "#PWR0169"

Commit message: LED 3V3x rename
Connections:
- net +3V3aa is gone; now on net +3V3d: R132.2
- net +3V3bb is gone; now on net +3V3e: R142.2
- net +3V3cc is gone; now on net +3V3f: R152.2
Changed lines of the file:
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@@
 			)
 		)
-		(property "Value" "+3V3bb"
+		(property "Value" "+3V3e"
 			(at 335.28 279.4 0)
+			(do_not_autoplace yes)
 			(effects
 				(font
@@
 			)
 		)
-		(property "Value" "+3V3cc"
+		(property "Value" "+3V3f"
 			(at 524.51 280.67 0)
+			(do_not_autoplace yes)
 			(effects
 				(font
@@
 			)
 		)
-		(property "Value" "+3V3aa"
+		(property "Value" "+3V3d"
 			(at 163.83 275.59 0)
+			(do_not_autoplace yes)
 			(effects
 				(font
