File: PCB/4 Layer nvme Carrier all M2/BIOS.kicad_sch (KiCad schematic)
At the start: 11 parts, among them U79 W25Q128JVSIQ

Commit message: first all-M.2 version
Other:
- title: (none) -> nvme Carrier for LattePanda Mu
Changed lines of the file:
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@@
 	(generator_version "8.0")
 	(paper "A4")
+	(title_block
+		(title "nvme Carrier for LattePanda Mu")
+		(date "2024-07-13")
+		(rev "V1.0")
+	)
 	(junction
 		(at 180.34 74.93)
