File: PCB/4 Layer nvme Carrier all M2/Ethernet.kicad_sch (KiCad schematic)
At the start: 28 parts, among them J6 RJ45_RB1-125B8G1A, U6 RTL8111H-CG-RH, U7 ULC0524P, U8 ULC0524P, Y1 25MHz

Commit message: first all-M.2 version
Other:
- title: Primer Carrier for LattePanda Mu -> nvme Carrier for LattePanda Mu
- moved on the sheet: C33, C34, C35, C36, C37, C38, C39, C40, C41, C42, C43, C44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
