File: PCB/4 Layer nvme Carrier all M2/LattePanda Module.kicad_sch (KiCad schematic)
At the start: 12 parts, among them J1 Conn_01x03_Pin, J11 Conn_01x03_Pin

Commit message: first all-M.2 version
Parts:
- H5, H6: value MountingHole_Pad -> MountingHole_Pad_50; LCSC Part # (none) -> C5301799; MPN (none) -> SMTWEM250STR
Connections:
- net USB_2_P5-: now reaches A1.109 (USB2_P5-)
- net USB_2_P5+: now reaches A1.111 (USB2_P5+)
- net SUSCLK: now reaches A1.131 (SUSCLK)
- net USB_2_P7+: now reaches A1.76 (USB2_P7+)
- net USB_2_P7-: now reaches A1.78 (USB2_P7-)
- net USB_2_P8+: now reaches A1.82 (USB2_P8+)
- net USB_2_P8-: now reaches A1.84 (USB2_P8-)
- net +12V renamed VDC
- no-connect marks 84 -> 77
Changed lines of the file:
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@@
 	)
 	(no_connect
-		(at 351.79 147.32)
-	)
-	(no_connect
 		(at 351.79 180.34)
 	)
@@
 	)
 	(no_connect
-		(at 270.51 195.58)
-	)
-	(no_connect
 		(at 351.79 134.62)
 	)
@@
 	)
 	(no_connect
-		(at 351.79 119.38)
-	)
-	(no_connect
 		(at 270.51 297.18)
 	)
@@
 	)
 	(no_connect
-		(at 270.51 200.66)
-	)
-	(no_connect
 		(at 351.79 269.24)
 	)
 	(no_connect
-		(at 270.51 198.12)
-	)
-	(no_connect
-		(at 270.51 203.2)
-	)
-	(no_connect
 		(at 351.79 271.78)
 	)
@@
 	)
 	(no_connect
-		(at 351.79 116.84)
-	)
-	(no_connect
 		(at 270.51 317.5)
 	)
@@
 	(wire
 		(pts
+			(xy 351.79 147.32) (xy 369.57 147.32)
+		)
+		(stroke
+			(width 0)
+			(type default)
+		)
+	)
+	(wire
+		(pts
 			(xy 238.76 172.72) (xy 270.51 172.72)
 		)
@@
 	(wire
 		(pts
+			(xy 238.76 195.58) (xy 270.51 195.58)
+		)
+		(stroke
+			(width 0)
+			(type default)
+		)
+	)
+	(wire
+		(pts
 			(xy 351.79 97.79) (xy 369.57 97.79)
 		)
@@
 	(wire
 		(pts
+			(xy 238.76 200.66) (xy 270.51 200.66)
+		)
+		(stroke
+			(width 0)
+			(type default)
+		)
+	)
+	(wire
+		(pts
 			(xy 238.76 139.7) (xy 270.51 139.7)
 		)
@@
 	(wire
 		(pts
+			(xy 351.79 116.84) (xy 363.22 116.84)
+		)
+		(stroke
+			(width 0)
+			(type default)
+		)
+	)
+	(wire
+		(pts
 			(xy 238.76 254) (xy 266.7 254)
 		)
@@
 	(wire
 		(pts
+			(xy 238.76 198.12) (xy 270.51 198.12)
+		)
+		(stroke
+			(width 0)
+			(type default)
+		)
+	)
+	(wire
+		(pts
 			(xy 215.9 73.66) (xy 270.51 73.66)
 		)
@@
 	(wire
 		(pts
+			(xy 351.79 119.38) (xy 363.22 119.38)
+		)
+		(stroke
+			(width 0)
+			(type default)
+		)
+	)
+	(wire
+		(pts
 			(xy 238.76 259.08) (xy 270.51 259.08)
 		)
@@
 	(wire
 		(pts
+			(xy 238.76 203.2) (xy 270.51 203.2)
+		)
+		(stroke
+			(width 0)
+			(type default)
+		)
+	)
+	(wire
+		(pts
 			(xy 304.8 38.1) (xy 304.8 44.45)
 		)
@@
 		)
 	)
+	(hierarchical_label "SUSCLK"
+		(shape input)
+		(at 369.57 147.32 0)
+		(effects
+			(font
+				(size 1.27 1.27)
+			)
+			(justify left)
+		)
+	)
 	(hierarchical_label "FAN_1_TAC"
 		(shape input)
@@
 		)
 	)
+	(hierarchical_label "USB_2_P7-"
+		(shape bidirectional)
+		(at 238.76 198.12 180)
+		(effects
+			(font
+				(size 1.27 1.27)
+			)
+			(justify right)
+		)
+	)
 	(hierarchical_label "REFCLK2+"
 		(shape output)
@@
 		)
 	)
+	(hierarchical_label "USB_2_P8+"
+		(shape bidirectional)
+		(at 238.76 200.66 180)
+		(effects
+			(font
+				(size 1.27 1.27)
+			)
+			(justify right)
+		)
+	)
 	(hierarchical_label "REFCLK3-"
 		(shape output)
@@
 		)
 	)
+	(hierarchical_label "USB_2_P5-"
+		(shape bidirectional)
+		(at 363.22 119.38 0)
+		(effects
+			(font
+				(size 1.27 1.27)
+			)
+			(justify left)
+		)
+	)
 	(hierarchical_label "TCP_0_HPD"
 		(shape input)
@@
 		)
 	)
+	(hierarchical_label "USB_2_P7+"
+		(shape bidirectional)
+		(at 238.76 195.58 180)
+		(effects
+			(font
+				(size 1.27 1.27)
+			)
+			(justify right)
+		)
+	)
 	(hierarchical_label "HSIO_11_TX-"
 		(shape output)
@@
 		)
 	)
+	(hierarchical_label "USB_2_P8-"
+		(shape bidirectional)
+		(at 238.76 203.2 180)
+		(effects
+			(font
+				(size 1.27 1.27)
+			)
+			(justify right)
+		)
+	)
 	(hierarchical_label "HSIO_0_TX+"
 		(shape output)
@@
 		)
 	)
+	(hierarchical_label "USB_2_P5+"
+		(shape bidirectional)
+		(at 363.22 116.84 0)
+		(effects
+			(font
+				(size 1.27 1.27)
+			)
+			(justify left)
+		)
+	)
 	(hierarchical_label "HSIO_6_RX+"
 		(shape input)
@@
 			)
 		)
-		(property "Value" "MountingHole_Pad"
+		(property "Value" "MountingHole_Pad_50"
 			(at 416.56 299.72 0)
 			(effects
@@
 			)
 		)
-		(property "Datasheet" "~"
+		(property "Datasheet" "https://www.lcsc.com/datasheet/lcsc_datasheet_2410121507_YIYUAN-SMTWEM250STR_C5301799.pdf"
 			(at 414.02 299.72 0)
 			(effects
@@
 			)
 		)
+		(property "LCSC Part #" "C5301799"
+			(at 414.02 299.72 0)
+			(effects
+				(font
+					(size 1.27 1.27)
+				)
+				(hide yes)
+			)
+		)
+		(property "MPN" "SMTWEM250STR"
+			(at 414.02 299.72 0)
+			(effects
+				(font
+					(size 1.27 1.27)
+				)
+				(hide yes)
+			)
+		)
 		(pin "1"
 		)
@@
 			)
 		)
-		(property "Value" "+12V"
+		(property "Value" "VDC"
 			(at 303.022 33.02 0)
 			(effects
@@
 			)
 		)
-		(property "Value" "MountingHole_Pad"
+		(property "Value" "MountingHole_Pad_50"
 			(at 441.96 299.72 0)
 			(effects
@@
 			)
 		)
-		(property "Datasheet" "~"
+		(property "Datasheet" "https://www.lcsc.com/datasheet/lcsc_datasheet_2410121507_YIYUAN-SMTWEM250STR_C5301799.pdf"
 			(at 439.42 299.72 0)
 			(effects
@@
 			(at 439.42 299.72 0)
 			(effects
+				(font
+					(size 1.27 1.27)
+				)
+				(hide yes)
+			)
+		)
+		(property "LCSC Part #" "C5301799"
+			(at 439.42 299.72 0)
+			(effects
+				(font
+					(size 1.27 1.27)
+				)
+				(hide yes)
+			)
+		)
+		(property "MPN" "SMTWEM250STR"
+			(at 439.42 299.72 0)
+			(effects
