File: PCB/4 Layer nvme Carrier all M2/M.2 M Key.kicad_sch (KiCad schematic)
At the start: 78 parts, among them J100 Bus_M.2_Socket_M, J110 Bus_M.2_Socket_M, J120 Bus_M.2_Socket_M, J130 Bus_M.2_Socket_M, J140 Bus_M.2_Socket_M, J150 Bus_M.2_Socket_M

Commit message: first all-M.2 version
Parts:
- H1032, H1042, H1080, H1130, H1142, H1180, H1230, H1242, H1280, H1330, H1342, H1380, H1430, H1442, H1480, H1530, H1542, H1580: value MountingHole_M2.5 -> MountingHole_Pad_15; footprint MountingHole:MountingHole_2.7mm_M2.5_DIN965_Pad_TopBottom -> A_HDJ_Library:MountingHole_3mm_M2_Pad_TopOnly; LCSC Part # (none) -> C5221852; MPN (none) -> SMTWEM215STR
