File: PCB/4 Layer nvme Carrier all M2/USB.kicad_sch (KiCad schematic)
At the start: 18 parts, among them J2 USB_A_Stacked, J3 USB3_A, J78 USB_A, U3 ULC0524P, U4 ULC0524P

Commit message: first all-M.2 version
Parts:
- added C130: 22uF/10V, A_HDJ_Library:C_0603_1608Metric, symbol Device:C
- added F79: 6V/1A, A_HDJ_Library:Fuse_0805_2012Metric, symbol Device:Fuse
- added J83: PINHD_2x5_Male, Connector_PinHeader_2.54mm:PinHeader_2x05_P2.54mm_Vertical, symbol PCM_SL_Pin_Headers:PINHD_2x5_Male
- added U84: ULC0524P, A_HDJ_Library:Diodes_UDFN-10_1.0x2.5mm_P0.5mm, symbol Power_Protection:D3V3XA4B10LP
Connections:
- net GND: now also C130.1, J83.7, J83.8, U84.3 (VSS), U84.8 (VSS)
- net +5V renamed +5Va
- net +5Va: now also C130.2, F79.1
- new net: F79.2, J83.1, J83.2
- new net USB_2_P5+: J83.5, U84.1, U84.10 (NC)
- new net USB_2_P5-: J83.3, U84.2, U84.9 (NC)
- new net USB_2_P6+: J83.6, U84.4, U84.7 (NC)
- new net USB_2_P6-: J83.4, U84.5, U84.6 (NC)
- no-connect marks 0 -> 2
Other:
- moved on the sheet: C28, C29, C30, C32, C88, D5, D6, D79, D80, F2, F3, F5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
