File: PCB/4 Layer nvme Carrier all M2/fan_temp.kicad_sch (KiCad schematic)
At the start: 20 parts, among them M1 Fan_4pin, M2 Fan_4pin

Commit message: first all-M.2 version
Parts:
- removed R73: 0R/1%, RES0603, symbol Device:R
- added C129: 100nF/50V, A_HDJ_Library:C_0402_1005Metric, symbol Device:C
- added D28: 1N5819WS, A_HDJ_Library:D_SOD-323, symbol Diode:1N5819WS
- added M3: Fan_4pin, Connector:FanPinHeader_1x04_P2.54mm_Vertical, symbol Motor:Fan_4pin
- added R107, R110: 4.7K/1%, A_HDJ_Library:R_0402_1005Metric, symbol Device:R
- added R108, R75: 21.5K/1%, A_HDJ_Library:R_0402_1005Metric, symbol Device:R
- added R109: 100R/1%, A_HDJ_Library:R_0402_1005Metric, symbol Device:R
Connections:
- net +3V3: now also R107.1
- net +5V: now also C129.1, D28.1 (K), M3.2 (+), R110.1
- net FAN_2_PWM: now also R107.2, R109.1
- net FAN_2_TAC: now also R108.1, R75.1; no longer R67.1, R70.1
- net GND: now also C129.2, M3.1 (-), R108.2
- new net: D28.2 (A), M3.3 (Tacho), R110.2, R75.2
- new net: M3.4 (PWM), R109.2
- new net: R67.1, R70.1
- no-connect marks 0 -> 2
Other:
- note added: "SYS FAN_12"
- note added: "SYS FAN_5"
- note removed: "SYS FAN"
- moved on the sheet: C84, C85, D26, D27, JP2, M1, M2, R63, R64, R65, R66, R67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
