File: PCB/4 Layer nvme Carrier all M2/nvme Carrier all M2.kicad_sch (KiCad schematic)
At the start: 8 parts

Commit message: first all-M.2 version
Parts:
- H71, H72, H73, H74: now fitted
Other:
- sheet LattePanda Module ports: added SUSCLK, USB_2_P5+, USB_2_P5-, USB_2_P7+, USB_2_P7-, USB_2_P8+, USB_2_P8-; removed none
- sheet M.2 E&M-Key ports: added SUSCLK, USB_2_P5+, USB_2_P5-; removed none
- sheet USB ports: added USB_2_P5+, USB_2_P5-, USB_2_P6+, USB_2_P6-; removed none
